File: kicad/bldcdriver/bldcdriver.kicad_pcb (KiCad board)
At the start: 2 copper layers, 68.6 x 33 mm, 39 parts, among them J1 Conn_01x04_Pin, J2 Conn_01x01_Pin, J3 Conn_01x01_Pin, J4 Conn_01x01_Pin, J5 Conn_01x04_Pin, J6 Conn_01x04_Pin, J7 Conn_01x04_Pin, J8 Conn_01x01_Pin, J9 Conn_01x01_Pin, U1 IRS2008S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

Commit message: finish
Parts:
- added D4: LED, LED_SMD:LED_0603_1608Metric, F.Cu at (171.4, 81.6)
- added D5: LED, LED_SMD:LED_0603_1608Metric, F.Cu at (171.4, 83.3)
- added D6: LED, LED_SMD:LED_0603_1608Metric, F.Cu at (171.5, 91.3)
- added D7: LED, LED_SMD:LED_0603_1608Metric, F.Cu at (171.6, 93.0)
- added D8: LED, LED_SMD:LED_0603_1608Metric, F.Cu at (171.4, 102.5)
- added D9: LED, LED_SMD:LED_0603_1608Metric, F.Cu at (171.4, 104.1)
- added R7: 4.7k, Resistor_SMD:R_0603_1608Metric_Pad0.98x0.95mm_HandSolder, F.Cu at (175.6, 85.0)
- added R8: 4.7k, Resistor_SMD:R_0603_1608Metric_Pad0.98x0.95mm_HandSolder, F.Cu at (175.6, 96.1)
- added R9: 4.7k, Resistor_SMD:R_0603_1608Metric_Pad0.98x0.95mm_HandSolder, F.Cu at (175.6, 100.0)
Routing:
- net Net-(D6-K): track 0.00 -> 5.72 mm
- net Net-(D8-K): track 0.00 -> 5.12 mm
- net Net-(D4-K): track 0.00 -> 4.84 mm
- net out_l: track 14.7 -> 18.6 mm
- net out_w: track 13.2 -> 17.0 mm
- net out_u: track 13.7 -> 17.4 mm
Other:
- board text added: "BLDC MD V1(alpha)"
- board text added: "L"
- board text added: "U"
- board text added: "W"
- board text added: "photo coupler register 5V-500Ω 3.3v-330Ω"
