File: kicad/bldcdriver/bldcdriver.kicad_sch (KiCad schematic)
At the start: 36 parts, among them J1 Conn_01x04_Pin, J2 Conn_01x01_Pin, J3 Conn_01x01_Pin, J4 Conn_01x01_Pin, J5 Conn_01x04_Pin, J6 Conn_01x04_Pin, J7 Conn_01x04_Pin, J8 Conn_01x01_Pin, J9 Conn_01x01_Pin, U1 IRS2008S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

Commit message: finish
Parts:
- added D4, D5, D6, D7, D8, D9: LED, LED_SMD:LED_0603_1608Metric, symbol Device:LED
- added R7, R8, R9: 4.7k, Resistor_SMD:R_0603_1608Metric_Pad0.98x0.95mm_HandSolder, symbol Device:R
Connections:
- net GND: now also D4.2 (A), D5.1 (K), D6.2 (A), D7.1 (K), D8.2 (A), D9.1 (K)
- net out_l: now also R9.1
- net out_u: now also R7.1
- net out_w: now also R8.1
- new net: D8.1 (K), D9.2 (A), R9.2
- new net: D6.1 (K), D7.2 (A), R8.2
- new net: D4.1 (K), D5.2 (A), R7.2
