File: kicad/MDhub/MDhub.kicad_pcb (KiCad board)
At the start: 2 copper layers, 83.8 x 52.1 mm, 49 parts, among them J1 USB_C_Receptacle_USB2.0_14P, J10 Conn_01x04_Pin, J11 Conn_01x02_Pin, J12 Conn_01x04_Pin, J13 Conn_01x03_Pin, J14 Conn_01x03_Pin, J15 Conn_01x03_Pin, J16 Conn_01x03_Pin, J17 Conn_01x05_Pin, J18 Conn_01x05_Pin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

Commit message: perf MDhub circuit
Parts:
- added LED3: LED, LED_SMD:LED_0603_1608Metric_Pad1.05x0.95mm_HandSolder, F.Cu at (223.5, 71.1)
- added LED4: LED, LED_SMD:LED_0603_1608Metric_Pad1.05x0.95mm_HandSolder, F.Cu at (223.5, 69.6)
- added R10: 165, Resistor_SMD:R_0603_1608Metric_Pad0.98x0.95mm_HandSolder, F.Cu at (222.5, 66.8)
- added R9: 165, Resistor_SMD:R_0603_1608Metric_Pad0.98x0.95mm_HandSolder, F.Cu at (220.7, 70.1)
- moved C4 4.49 mm to (221.0, 74.7), turned to 90 degrees
Routing:
- net PB5: track 0.00 -> 8.77 mm, vias 0 -> 1
- net PB4: track 0.00 -> 8.41 mm, vias 0 -> 1
- net CAN_RX: track 43.8 -> 36.3 mm
- net VBUS: track 185.6 -> 182.5 mm
- net Net-(LED3-K): track 0.00 -> 1.96 mm
- net Net-(LED4-K): track 0.00 -> 1.94 mm
- net Vbat: track 103.6 -> 102.5 mm
- net GND: vias 14 -> 107

Commit message: mdhub
Parts:
- removed LED3, LED4: LED, LED_SMD:LED_0603_1608Metric_Pad1.05x0.95mm_HandSolder
- added D1: WS2812B, LED_SMD:LED_WS2812B_PLCC4_5.0x5.0mm_P3.2mm, F.Cu at (249.5, 79.2)
- added J21: Conn_01x05_Pin, Connector_Molex:Molex_KK-254_AE-6410-05A_1x05_P2.54mm_Vertical, F.Cu at (254.8, 94.3)
- added J22: Conn_01x05_Pin, Connector_Molex:Molex_KK-254_AE-6410-05A_1x05_P2.54mm_Vertical, F.Cu at (212.8, 94.3)
- added J23: Conn_01x02_Pin, Connector_Hirose:Hirose_DF13-02P-1.25DS_1x02_P1.25mm_Horizontal, F.Cu at (261.9, 66.5)
- added J24: Conn_01x02_Pin, Connector_Hirose:Hirose_DF13-02P-1.25DS_1x02_P1.25mm_Horizontal, F.Cu at (261.9, 71.9)
- added J25: Conn_01x05_Pin, Connector_Molex:Molex_KK-254_AE-6410-05A_1x05_P2.54mm_Vertical, F.Cu at (256.2, 73.6)
- added SW2: SW_Wuerth_450301014042, Button_Switch_THT:SW_Slide-03_Wuerth-WS-SLTV_10x2.5x6.4_P2.54mm, F.Cu at (179.6, 99.3)
- added SW3: SW_Wuerth_450301014042, Button_Switch_THT:SW_Slide-03_Wuerth-WS-SLTV_10x2.5x6.4_P2.54mm, F.Cu at (243.2, 71.7)
- added U3: SOP-J8, footprints2:SOP-J8, B.Cu at (204.0, 100.6)
- C11, C12, C3, C7, L1, R2, R3, R7: moved to F.Cu
- J13, J16: value Conn_01x03_Pin -> Conn_01x04_Pin; footprint Connector_Molex:Molex_KK-254_AE-6410-03A_1x03_P2.54mm_Vertical -> Connector_Hirose:Hirose_DF13-04P-1.25DSA_1x04_P1.25mm_Vertical
- J14, J15: value Conn_01x03_Pin -> Conn_01x02_Pin; footprint Connector_Molex:Molex_KK-254_AE-6410-03A_1x03_P2.54mm_Vertical -> Connector_Hirose:Hirose_DF13-02P-1.25DS_1x02_P1.25mm_Horizontal
- R10: value 165 -> fuse
- R9: value 165 -> R; moved to B.Cu
- U1: moved to B.Cu
- moved R8 63.9 mm to (256.9, 55.1)
- moved SW1 60.8 mm to (249.2, 55.1)
- moved J6 54.0 mm to (212.8, 101.9), turned to 0 degrees
- moved U1 49.5 mm to (248.4, 61.5), turned to 0 degrees
- moved R9 47.9 mm to (182.8, 99.3), turned to 0 degrees
- moved J1 41.2 mm to (263.9, 84.8), turned to 90 degrees
- moved R10 39.7 mm to (256.3, 87.7), turned to 180 degrees
- moved C7 39.1 mm to (225.3, 89.2), turned to -90 degrees
- moved R7 38.9 mm to (226.8, 88.9), turned to 90 degrees
- moved J14 38.1 mm to (261.7, 55.8), turned to -90 degrees
- moved R1 37.0 mm to (256.3, 80.3)
- moved J16 36.8 mm to (214.3, 88.1)
- moved BOOT1 35.2 mm to (232.4, 88.6), turned to 180 degrees
- moved R5 34.1 mm to (250.6, 86.1), turned to 0 degrees
- moved LED2 33.6 mm to (250.6, 87.7)
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Connections:
- BOOT1 pad 1: BOOT0 -> Vbat
- BOOT1 pad 2: GND -> BOOT0
- C4 pad 1: VBUS -> Net-(DCDC1-STBY)
- C7 pad 1: BOOT0 -> GND
- C7 pad 2: GND -> BOOT0
- DCDC1 pad 1: VBUS -> Net-(DCDC1-STBY)
- DCDC1 pad 3: VBUS -> Net-(DCDC1-STBY)
- J1 pad A6: PA12 -> unconnected-(J1-D+-PadA6)
- J1 pad A7: PA11 -> unconnected-(J1-D--PadA7)
- J10 pad 1: unconnected-(J10-Pin_1-Pad1) -> VBUS
- J10 pad 2: PB6 -> PB10
- J10 pad 3: PB7 -> PB12
- J11 pad 1: VS -> GND1
- J11 pad 2: GND1 -> VS
- J12 pad 2: CAN_H -> CAN_H2
- J12 pad 3: CAN_L -> CAN_L2
- J13 pad 2: CH1_TIM3 -> INP5
- J13 pad 3: GND -> INP15
- J14 pad 1: VBUS -> CAN_H
- J14 pad 2: CH2_TIM3 -> CAN_L
- J15 pad 1: VBUS -> CAN_H
- J15 pad 2: ETR_TIM8 -> CAN_L
- J16 pad 2: INP1 -> CH1_TIM5
- J16 pad 3: GND -> CH2_TIM5
- J19 pad 1: VS -> GND1
- J19 pad 2: GND1 -> VS
- J20 pad 2: CAN_H -> CAN_H2
- J20 pad 3: CAN_L -> CAN_L2
- J6 pad 1: CH1_TIM8 -> CH1_TIM5
- J6 pad 3: CH2_TIM8 -> CH2_TIM5
- J6 pad 4: ETR_TIM8 -> ETR_TIM5
- J7 pad 1: VS -> GND1
- J7 pad 2: GND1 -> VS
- J8 pad 1: VS -> GND1
- J8 pad 2: GND1 -> VS
- J9 pad 1: unconnected-(J9-Pin_1-Pad1) -> VBUS
- J9 pad 2: PB6 -> PB10
- J9 pad 3: PB7 -> PB12
- R1 pad 1: Net-(J1-VBUS-PadA4) -> VBUS
- R1 pad 2: VBUS -> Net-(DCDC1-STBY)
- R10 pad 1: Net-(LED4-K) -> Net-(J1-VBUS-PadA4)
- R10 pad 2: GND -> VBUS
- R7 pad 1: Vbat -> BOOT0
- R7 pad 2: BOOT0 -> GND
- R9 pad 2: GND -> CAN_L2
- U1 pad 1: CAN_TX -> CAN1_TX
- U1 pad 4: CAN_RX -> CAN1_RX
- U2 pad 10: ETR_TIM8 -> CH1_TIM5
- U2 pad 11: INP1 -> CH2_TIM5
- U2 pad 13: PA3 -> INP15
- U2 pad 14: PA4 -> ETR_TIM5
- U2 pad 19: PB1 -> INP5
- U2 pad 21: CH1_TIM8 -> PB10
- U2 pad 25: CAN_RX -> PB12
- U2 pad 26: CH2_TIM8 -> PB13
- U2 pad 31: CAN_TX -> CH3_TIM1
- U2 pad 33: PA12 -> ETR_TIM1
- U2 pad 34: SWCLK -> SWDIO
- U2 pad 37: SWDIO -> SWCLK
- U2 pad 41: PB5 -> CAN2_RX
- U2 pad 42: PB6 -> CAN2_TX
- U2 pad 43: PB7 -> CAN1_TX
- U2 pad 45: PB8 -> CAN1_RX
Routing:
- net VBUS: track 182.5 -> 246.2 mm, vias 2 -> 0
- net Net-(DCDC1-STBY): track 0.00 -> 45.4 mm
- net PB12: track 0.00 -> 43.8 mm, vias 0 -> 1
- net CAN_TX: track 40.5 -> 0.00 mm, vias 1 -> 0
- net CAN2_RX: track 0.00 -> 38.7 mm
- net PB10: track 0.00 -> 37.9 mm, vias 0 -> 1
- net ETR_TIM8: track 37.8 -> 0.00 mm
- net ETR_TIM1: track 0.00 -> 37.1 mm
- net CAN_RX: track 36.3 -> 0.00 mm, vias 1 -> 0
- net CAN2_TX: track 0.00 -> 34.5 mm
- net CAN1_RX: track 0.00 -> 33.6 mm, vias 0 -> 4
- net CH1_TIM5: track 0.00 -> 33.3 mm, vias 0 -> 1
- net CH2_TIM8: track 32.0 -> 0.00 mm
- net CH2_TIM5: track 0.00 -> 31.9 mm
- net CAN_H2: track 0.00 -> 31.8 mm
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- added copper zone on B.Cu, net GND1
- added copper zone on F.Cu, net VS
- removed copper zone on F.Cu, net GND1
- removed copper zone on B.Cu, net VS
Other:
- board size 83.8 x 52.1 mm -> 89.2 x 52.1 mm

Commit message: hattyuuzumi
Parts:
- added G***: LOGO, _gazou:core, F.Cu at (202.7, 71.6)
- added G***: LOGO, _gazou:full, F.Cu at (196.5, 71.0)
- added H1: MountingHole, MountingHole:MountingHole_3.2mm_M3, F.Cu at (250.2, 86.0)
- added H2: MountingHole, MountingHole:MountingHole_3.2mm_M3, F.Cu at (263.1, 57.8)
- added H3: MountingHole, MountingHole:MountingHole_3.2mm_M3, F.Cu at (181.2, 99.4)
- added H4: MountingHole, MountingHole:MountingHole_3.2mm_M3, F.Cu at (182.1, 57.8)
- R5, R8: moved to B.Cu
- moved C4 34.6 mm to (255.0, 76.2)
- moved R4 29.2 mm to (245.5, 74.1), turned to 90 degrees
- moved LED1 29.1 mm to (247.1, 74.1), turned to 90 degrees
- moved DCDC1 29.0 mm to (249.7, 74.4), turned to 90 degrees
- moved C3 25.5 mm to (249.3, 71.7), turned to 0 degrees
- moved LED2 17.5 mm to (251.1, 70.1)
- moved R5 15.0 mm to (250.2, 71.0), turned to -90 degrees
- moved R8 7.24 mm to (250.1, 57.5)
- moved J7 7.17 mm to (204.5, 61.0), turned to 180 degrees
- moved J8 7.17 mm to (204.5, 81.3), turned to 180 degrees
- moved R9 6.83 mm to (189.6, 99.3)
- moved SW2 6.83 mm to (186.3, 98.2)
- moved J11 6.16 mm to (190.3, 67.1)
- moved J14 6.04 mm to (256.3, 58.4), turned to 0 degrees
- moved J20 5.97 mm to (197.2, 94.7)
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Connections:
- J25 pad 2: SPI_MOSI -> SPI_MOSI2
- SW3 pad 1: SPI_MOSI -> PB15
- SW3 pad 2: PB15 -> SPI_MOSI2
Routing:
- net VBUS: track 246.2 -> 212.0 mm, vias 0 -> 1
- net Net-(DCDC1-STBY): track 45.4 -> 11.9 mm
- net SPI_MOSI2: track 0.00 -> 13.8 mm
- net SPI_MOSI: track 13.3 -> 0.00 mm
- net Vbat: track 78.7 -> 88.3 mm, vias 7 -> 9
- net CAN_H: track 44.5 -> 38.7 mm, vias 0 -> 1
- net Net-(SW1-B): track 7.90 -> 2.48 mm
- net PB15: track 16.9 -> 11.9 mm, vias 0 -> 1
- net CAN_L: track 40.0 -> 36.4 mm, vias 0 -> 1
- net ETR_TIM5: track 29.5 -> 32.1 mm
- net CAN_H2: track 31.8 -> 29.4 mm
- net NRST: track 30.6 -> 32.9 mm, vias 6 -> 4
- net CAN_L2: track 26.5 -> 24.4 mm
- net CAN1_TX: track 31.4 -> 29.5 mm, vias 4 -> 2
- net CAN1_RX: track 33.6 -> 31.8 mm, vias 4 -> 2
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Other:
- board text added: "5V"
- board text added: "5V 1 2 3 G"
- board text added: "A 5V B Z G"
- board text added: "GND"
- board text added: "LED"
- board text added: "MDhub(wide cover) x4 Encoder or hole sensor x2 CANFD x2 I2C slot x1 SPI"
- board text added: "OUT"
- board text added: "PA3"
- board text added: "PB1"
- board text added: "Ron"
- board text added: "SCL"
- board text added: "SDA"
- board text added: "TIM1"
- board text added: "TIM2"
- board text added: "TIM3"
- board text added: "TIM5"
- board text added: "Vcc"
- board text added: "t5ch1"
- board text added: "t5ch2"
