File: kicad/MDhub/MDhub.kicad_sch (KiCad schematic)
At the start: 49 parts, among them J1 USB_C_Receptacle_USB2.0_14P, J10 Conn_01x04_Pin, J11 Conn_01x02_Pin, J12 Conn_01x04_Pin, J13 Conn_01x03_Pin, J14 Conn_01x03_Pin, J15 Conn_01x03_Pin, J16 Conn_01x03_Pin, J17 Conn_01x05_Pin, J18 Conn_01x05_Pin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

Commit message: perf MDhub circuit
Parts:
- added LED3, LED4: LED, LED_SMD:LED_0603_1608Metric_Pad1.05x0.95mm_HandSolder, symbol Device:LED
- added R10, R9: 165, Resistor_SMD:R_0603_1608Metric_Pad0.98x0.95mm_HandSolder, symbol Device:R
Connections:
- net GND: now also R10.2, R9.2
- net PB4: now also LED3.2 (A)
- net PB5: now also LED4.2 (A)
- new net: LED4.1 (K), R10.1
- new net: LED3.1 (K), R9.1
Other:
- moved on the sheet: J17, J18

Commit message: finish
Changed lines of the file:
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@@
 (kicad_sch
-	(version 20231120)
+	(version 20250114)
 	(generator "eeschema")
-	(generator_version "8.0")
+	(generator_version "9.0")
 	(paper "A4")

Commit message: mdhub
Parts:
- removed J13, J14, J15, J16: Conn_01x03_Pin, Connector_Molex:Molex_KK-254_AE-6410-03A_1x03_P2.54mm_Vertical, symbol Connector:Conn_01x03_Pin
- removed LED3, LED4: LED, LED_SMD:LED_0603_1608Metric_Pad1.05x0.95mm_HandSolder, symbol Device:LED
- added D1: WS2812B, LED_SMD:LED_WS2812B_PLCC4_5.0x5.0mm_P3.2mm, symbol LED:WS2812B
- added J13, J16: Conn_01x04_Pin, Connector_Hirose:Hirose_DF13-04P-1.25DSA_1x04_P1.25mm_Vertical, symbol Connector:Conn_01x04_Pin
- added J14, J15, J23, J24: Conn_01x02_Pin, Connector_Hirose:Hirose_DF13-02P-1.25DS_1x02_P1.25mm_Horizontal, symbol Connector:Conn_01x02_Pin
- added J21, J22, J25: Conn_01x05_Pin, Connector_Molex:Molex_KK-254_AE-6410-05A_1x05_P2.54mm_Vertical, symbol Connector:Conn_01x05_Pin
- added SW2, SW3: SW_Wuerth_450301014042, Button_Switch_THT:SW_Slide-03_Wuerth-WS-SLTV_10x2.5x6.4_P2.54mm, symbol Switch:SW_Wuerth_450301014042
- added U3: SOP-J8, footprints2:SOP-J8, symbol 2025-05-15_08-12-01:SOP-J8
- R10: value 165 -> fuse
- R9: value 165 -> R
Connections:
- net INP1 is gone; now on net CH2_TIM5: U2.11 (PA1)
- net PA4 is gone; now on net ETR_TIM5: U2.14 (PA4)
- net PB8 is gone; now on net CAN1_RX: U2.45 (PB8)
- net +3V3: now also BOOT1.1; no longer R7.1
- net BOOT0: now also BOOT1.2, C7.2, R7.1; no longer BOOT1.1, C7.1, R7.2
- net CAN_H: now also J14.1 (Pin_1), J15.1 (Pin_1), J23.1 (Pin_1), J24.1 (Pin_1); no longer J12.2 (Pin_2), J20.2 (Pin_2)
- net CAN_L: now also J14.2 (Pin_2), J15.2 (Pin_2), J23.2 (Pin_2), J24.2 (Pin_2); no longer J12.3 (Pin_3), J20.3 (Pin_3)
- net CH1_TIM1: now also J21.2 (Pin_2)
- net CH2_TIM1: now also J21.3 (Pin_3)
- net CH3_TIM2: now also J22.4 (Pin_4)
- net ETR_TIM1: now also U2.33 (PA12)
- net GND: now also C7.1, R7.2, D1.3 (VSS), J13.4 (Pin_4), J16.4 (Pin_4), J21.5 (Pin_5), J22.5 (Pin_5), J25.5 (Pin_5), U3.2 (GND), U3.8 (STB); no longer BOOT1.2, C7.2, R10.2, R9.2
- net GND1: now also J11.1 (Pin_1), J19.1 (Pin_1), J7.1 (Pin_1), J8.1 (Pin_1); no longer J11.2 (Pin_2), J19.2 (Pin_2), J7.2 (Pin_2), J8.2 (Pin_2)
- net PA11: no longer J1.A7 (D-), J1.B7 (D-)
- net PB14: now also J25.3 (Pin_3)
- net PB15: now also SW3.2 (C)
- net PB2: now also J25.4 (Pin_4)
- net SWCLK: now also U2.37 (PA14(JTCK); no longer U2.34 (PA13(JTMS)
- net SWDIO: now also U2.34 (PA13(JTMS); no longer U2.37 (PA14(JTCK)
- net VBUS: now also J10.1 (Pin_1), J9.1 (Pin_1), R1.1, R10.2, D1.1 (VDD), J13.1 (Pin_1), J16.1 (Pin_1), J21.1 (Pin_1), J22.1 (Pin_1), J25.1 (Pin_1), U3.3 (VCC); no longer C4.1, DCDC1.1 (VIN), DCDC1.3 (STBY), R1.2
- net VS: now also J11.2 (Pin_2), J19.2 (Pin_2), J7.2 (Pin_2), J8.2 (Pin_2); no longer J11.1 (Pin_1), J19.1 (Pin_1), J7.1 (Pin_1), J8.1 (Pin_1)
- net at R10.1: now also J1.A4 (VBUS), J1.A9 (VBUS), J1.B4 (VBUS), J1.B9 (VBUS)
- net at R9.1: now also SW2.1 (B)
- net CAN_RX renamed CAN1_RX
- net CAN1_RX: no longer U2.25 (PB12)
- net CAN_TX renamed CAN1_TX
- net CAN1_TX: now also U2.43 (PB7); no longer U2.31 (PA10)
- net CH1_TIM8 renamed CH1_TIM5
- net CH1_TIM5: now also U2.10 (PA0), J16.2 (Pin_2), J22.2 (Pin_2); no longer U2.21 (PB10)
- net CH2_TIM8 renamed CH2_TIM5
- net CH2_TIM5: now also J16.3 (Pin_3), J22.3 (Pin_3); no longer U2.26 (PB13)
- net ETR_TIM8 renamed ETR_TIM5
- net ETR_TIM5: no longer U2.10 (PA0)
- removed net PA12: J1.A6 (D+), J1.B6 (D+), U2.33 (PA12)
- net PA3 renamed INP15
- net INP15: now also J13.3 (Pin_3)
- net PB1 renamed INP5
- net INP5: now also J13.2 (Pin_2)
- net PB5 renamed CAN2_RX
- net CAN2_RX: now also U3.4 (RXD)
- net PB6 renamed PB10
- net PB10: now also U2.21 (PB10); no longer U2.42 (PB6)
- net PB7 renamed PB12
- net PB12: now also U2.25 (PB12); no longer U2.43 (PB7)
- new net: D1.4 (DIN), SW3.3 (A)
- new net: C4.1, DCDC1.1 (VIN), DCDC1.3 (STBY), R1.2
- new net CAN2_TX: U2.42 (PB6), U3.1 (TXD)
- new net CAN_H2: J12.2 (Pin_2), J20.2 (Pin_2), SW2.2 (C), U3.7 (CANH)
- new net CAN_L2: J12.3 (Pin_3), J20.3 (Pin_3), R9.2, U3.6 (CANL)
- new net CH3_TIM1: J21.4 (Pin_4), U2.31 (PA10)
- new net PB13: U2.26 (PB13)
- new net SPI_MOSI: J25.2 (Pin_2), SW3.1 (B)
Other:
- moved on the sheet: BOOT1, C4, C6, C7, J12, J2, J20, LED1, LED2, R1, R4, R5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

Commit message: hattyuuzumi
Parts:
- added H1, H2, H3, H4: MountingHole, MountingHole:MountingHole_3.2mm_M3, symbol Mechanical:MountingHole
Connections:
- net PB15: now also SW3.1 (B); no longer SW3.2 (C)
- net SPI_MOSI renamed SPI_MOSI2
- net SPI_MOSI2: now also SW3.2 (C); no longer SW3.1 (B)
