File: kicad/MDhubv2/Mdhubv2.kicad_sch (KiCad schematic)
At the start: 0 parts

Commit message: a
Parts:
- added U1: STM32G0B1CBTx, Package_QFP:LQFP-48_7x7mm_P0.5mm, symbol MCU_ST_STM32G0:STM32G0B1CBTx
Connections:
- new net CLK: U1.36 (PA14)
- new net DIO: U1.35 (PA13)
- new net GND: U1.7 (VSS)
- new net PA0: U1.11 (PA0)
- new net PA1: U1.12 (PA1)
- new net PA10: U1.32 (PA10/UCPD1_DBCC2)
- new net PA11: U1.33 (PA9/PA11)
- new net PA12: U1.34 (PA10/PA12)
- new net PA15: U1.37 (PA15)
- new net PA2: U1.13 (PA2)
- new net PA3: U1.14 (PA3)
- new net PA4: U1.15 (PA4)
- new net PA5: U1.16 (PA5)
- new net PA6: U1.17 (PA6)
- new net PA7: U1.18 (PA7)
- new net PA8: U1.28 (PA8)
- new net PA9: U1.29 (PA9/UCPD1_DBCC1)
- new net PB0: U1.19 (PB0)
- new net PB1: U1.20 (PB1)
- new net PB10: U1.22 (PB10)
- new net PB11: U1.23 (PB11)
- new net PB12: U1.24 (PB12)
- new net PB13: U1.25 (PB13)
- new net PB14: U1.26 (PB14)
- new net PB15: U1.27 (PB15)
- new net PB2: U1.21 (PB2)
- new net PB3: U1.42 (PB3)
- new net PB4: U1.43 (PB4)
- new net PB5: U1.44 (PB5)
- new net PB6: U1.45 (PB6)
- new net PB7: U1.46 (PB7)
- new net PB8: U1.47 (PB8)
- new net PB9: U1.48 (PB9)
- new net PC13: U1.1 (PC13)
- new net PC14: U1.2 (PC14)
- new net PC15: U1.3 (PC15)
- new net PC6: U1.30 (PC6)
- new net PC7: U1.31 (PC7)
- new net PD0: U1.38 (PD0)
- new net PD1: U1.39 (PD1)
- new net PD2: U1.40 (PD2)
- new net PD3: U1.41 (PD3)
- new net PF0: U1.8 (PF0)
- new net PF1: U1.9 (PF1)
- new net PF2: U1.10 (PF2)
- new net VDD: U1.4 (VBAT), U1.6 (VDD)
- new net VREF: U1.5 (VREF+)

Commit message: a
Parts:
- added BOOT1, RESET1: SW_Push, Button_Switch_SMD:SW_Tactile_SPST_NO_Straight_CK_PTS636Sx25SMTRLFS, symbol Switch:SW_Push
- added C1, C2, C3: 0.1u, symbol Device:C
- added C4: 10u(DFP, Capacitor_SMD:C_0603_1608Metric, symbol Device:C
- added C6, C7: 0.1u, Capacitor_SMD:C_0603_1608Metric, symbol Device:C
- added DCDC1: BU33TD3WG, footprints:SSOP5, symbol jisaku:Rohm_BU33TD3WG
- added J1: USB_C_Receptacle_USB2.0_14P, jisaku:USB_C_Receptacle_aitendo, symbol Connector:USB_C_Receptacle_USB2.0_14P
- added J12, J20: Conn_01x04_Pin, Connector_PinHeader_2.54mm:PinHeader_1x04_P2.54mm_Horizontal, symbol Connector:Conn_01x04_Pin
- added J14, J15, J23, J24: Conn_01x02_Pin, Connector_Hirose:Hirose_DF13-02P-1.25DS_1x02_P1.25mm_Horizontal, symbol Connector:Conn_01x02_Pin
- added J2: Conn_01x04_Pin, Connector_Molex:Molex_KK-254_AE-6410-04A_1x04_P2.54mm_Vertical, symbol Connector:Conn_01x04_Pin
- added L1: L, symbol Device:L
- added LED1, LED2: LED, LED_SMD:LED_0603_1608Metric_Pad1.05x0.95mm_HandSolder, symbol Device:LED
- added R1, R10: fuse, Resistor_SMD:R_0603_1608Metric_Pad0.98x0.95mm_HandSolder, symbol Device:R
- added R2, R3: 5.1k, Resistor_SMD:R_0603_1608Metric_Pad0.98x0.95mm_HandSolder, symbol Device:R
- added R4, R5: 165, Resistor_SMD:R_0603_1608Metric_Pad0.98x0.95mm_HandSolder, symbol Device:R
- added R6, R7: 10k, Resistor_SMD:R_0603_1608Metric_Pad0.98x0.95mm_HandSolder, symbol Device:R
- added R8, R9: R, Resistor_SMD:R_0603_1608Metric_Pad0.98x0.95mm_HandSolder, symbol Device:R
- added SW1, SW2: SW_Wuerth_450301014042, Button_Switch_THT:SW_Slide-03_Wuerth-WS-SLTV_10x2.5x6.4_P2.54mm, symbol Switch:SW_Wuerth_450301014042
- added U2, U3: SOP-J8, footprints2:SOP-J8, symbol 2025-05-15_08-12-01:SOP-J8
- added X1: IQXO-70, Oscillator:Oscillator_SMD_IQD_IQXO70-4Pin_7.5x5.0mm, symbol Oscillator:IQXO-70
Connections:
- net GND: now also C1.2, C2.2, C3.2, C4.2, C6.2, C7.1, DCDC1.2 (GND), J1.A1 (GND), J1.A12 (GND), J1.B1 (GND), J1.B12 (GND), J1.S1 (SHIELD), J12.4 (Pin_4), J2.4 (Pin_4), J20.4 (Pin_4), R2.1, R3.2, R4.2, R5.2, R7.2, RESET1.2, U2.2 (GND), U2.8 (STB), U3.2 (GND), U3.8 (STB), X1.2 (GND)
- net PA5: now also C6.1, R6.2, RESET1.1
- net VREF: now also C2.1, L1.1
- net PA0 renamed ADC0
- net PA1 renamed ADC1
- net PA2 renamed ADC2
- net PA3 renamed ADC3
- net PA4 renamed ADC4
- net PA6 renamed I2C_SDA
- net PA7 renamed I2C_SCL
- net PB12 renamed CAN2_RX
- net CAN2_RX: now also U3.4 (RXD)
- net PB13 renamed CAN2_TX
- net CAN2_TX: now also U3.1 (TXD)
- net PC13 renamed CS0
- net PC14 renamed CS1
- net PC15 renamed CS2
- net PD0 renamed CAN1_RX
- net CAN1_RX: now also U2.4 (RXD)
- net PD1 renamed CAN1_TX
- net CAN1_TX: now also U2.1 (TXD)
- net PF1 renamed CS3
- net PF2 renamed CS4
- net VDD renamed +3V3
- net +3V3: now also BOOT1.1, C1.1, C3.1, DCDC1.5 (VOUT), J2.1 (Pin_1), L1.2, LED1.2 (A), R6.1, X1.4 (V+)
- new net: R9.1, SW2.1 (B)
- new net: LED1.1 (K), R4.1
- new net: LED2.1 (K), R5.1
- new net: J1.A5 (CC1), R2.2
- new net: C4.1, DCDC1.1 (VIN), DCDC1.3 (STBY), R1.2
- new net: R8.1, SW1.1 (B)
- new net: J1.A4 (VBUS), J1.A9 (VBUS), J1.B4 (VBUS), J1.B9 (VBUS), R10.1
- new net: J1.B5 (CC2), R3.1
- new net BOOT0: BOOT1.2, C7.2, R7.1
- new net CAN_H: J14.1 (Pin_1), J15.1 (Pin_1), J23.1 (Pin_1), J24.1 (Pin_1), SW1.2 (C), U2.7 (CANH)
- new net CAN_H2: J12.2 (Pin_2), J20.2 (Pin_2), SW2.2 (C), U3.7 (CANH)
- new net CAN_L: J14.2 (Pin_2), J15.2 (Pin_2), J23.2 (Pin_2), J24.2 (Pin_2), R8.2, U2.6 (CANL)
- new net CAN_L2: J12.3 (Pin_3), J20.3 (Pin_3), R9.2, U3.6 (CANL)
- new net PH0: X1.3 (OUT)
- new net SWCLK: J2.3 (Pin_3)
- new net SWDIO: J2.2 (Pin_2)
- new net VBUS: J12.1 (Pin_1), J20.1 (Pin_1), LED2.2 (A), R1.1, R10.2, U2.3 (VCC), U3.3 (VCC)

Commit message: a
Parts:
- removed BOOT1, RESET1: SW_Push, Button_Switch_SMD:SW_Tactile_SPST_NO_Straight_CK_PTS636Sx25SMTRLFS, symbol Switch:SW_Push
- removed C6, C7: 0.1u, Capacitor_SMD:C_0603_1608Metric, symbol Device:C
- removed R1: fuse, Resistor_SMD:R_0603_1608Metric_Pad0.98x0.95mm_HandSolder, symbol Device:R
- removed R6, R7: 10k, Resistor_SMD:R_0603_1608Metric_Pad0.98x0.95mm_HandSolder, symbol Device:R
- added J10: Conn_01x04_Pin, Connector_Molex:Molex_KK-254_AE-6410-04A_1x04_P2.54mm_Vertical, symbol Connector:Conn_01x04_Pin
- added J11: Conn_01x02_Pin, Connector_Molex:Molex_KK-254_AE-6410-02A_1x02_P2.54mm_Vertical, symbol Connector:Conn_01x02_Pin
- added J13: Conn_01x04_Pin, Connector_PinHeader_2.54mm:PinHeader_1x04_P2.54mm_Vertical, symbol Connector:Conn_01x04_Pin
- added J16: Conn_01x02_Pin, Connector_PinSocket_2.54mm:PinSocket_1x02_P2.54mm_Vertical, symbol Connector:Conn_01x02_Pin
- added J17, J3, J4, J5, J6: Conn_01x05_Pin, Connector_JST:JST_XH_B5B-XH-A_1x05_P2.50mm_Vertical, symbol Connector:Conn_01x05_Pin
- added J18: Conn_01x03_Pin, Connector_PinHeader_2.54mm:PinHeader_1x03_P2.54mm_Vertical, symbol Connector:Conn_01x03_Pin
- added J19, J21: Conn_01x02_Pin, Connector_AMASS:AMASS_XT30U-F_1x02_P5.0mm_Vertical, symbol Connector:Conn_01x02_Pin
- added J22, J25: Conn_01x02_Pin, Connector_AMASS:AMASS_XT60PW-M_1x02_P7.20mm_Horizontal, symbol Connector:Conn_01x02_Pin
- added J26, J27, J28, J29, J30: Conn_01x03_Pin, Connector_JST:JST_XH_B3B-XH-A_1x03_P2.50mm_Vertical, symbol Connector:Conn_01x03_Pin
- added J7, J8: Conn_02x03_Counter_Clockwise, Connector_PinHeader_2.54mm:PinHeader_2x03_P2.54mm_Vertical, symbol Connector_Generic:Conn_02x03_Counter_Clockwise
- added J9: Conn_01x05_Pin, Connector_PinHeader_2.54mm:PinHeader_1x05_P2.54mm_Vertical, symbol Connector:Conn_01x05_Pin
- C1, C2, C3: footprint (none) -> Capacitor_SMD:C_0603_1608Metric
- J14, J15, J23, J24: footprint Connector_Hirose:Hirose_DF13-02P-1.25DS_1x02_P1.25mm_Horizontal -> Connector_JST:JST_XH_S2B-XH-A_1x02_P2.50mm_Horizontal
- L1: footprint (none) -> Inductor_SMD:L_0603_1608Metric
- SW1, SW2: footprint Button_Switch_THT:SW_Slide-03_Wuerth-WS-SLTV_10x2.5x6.4_P2.54mm -> jisaku:SW_Slide-03_Wuerth-WS-SLTV_10x2.5x6.4_P2.54mm
Connections:
- net PH0 is gone; now on net PF0: X1.3 (OUT)
- net SWCLK is gone; now on net CLK: J2.3 (Pin_3)
- net SWDIO is gone; now on net DIO: J2.2 (Pin_2)
- net +3V3: now also J10.1 (Pin_1), J13.1 (Pin_1), J17.1 (Pin_1), J26.1 (Pin_1), J27.1 (Pin_1), J28.1 (Pin_1), J29.1 (Pin_1), J30.1 (Pin_1), J7.1 (Pin_1), J8.1 (Pin_1)
- net ADC0: now also J28.2 (Pin_2)
- net ADC1: now also J29.2 (Pin_2)
- net ADC2: now also J30.2 (Pin_2)
- net ADC3: now also J27.2 (Pin_2)
- net ADC4: now also J26.2 (Pin_2)
- net CS0: now also J9.1 (Pin_1)
- net CS1: now also J9.2 (Pin_2)
- net CS2: now also J9.3 (Pin_3)
- net CS3: now also J9.4 (Pin_4)
- net CS4: now also J9.5 (Pin_5)
- net GND: now also J10.4 (Pin_4), J13.4 (Pin_4), J17.5 (Pin_5), J26.3 (Pin_3), J27.3 (Pin_3), J28.3 (Pin_3), J29.3 (Pin_3), J3.5 (Pin_5), J30.3 (Pin_3), J4.5 (Pin_5), J5.5 (Pin_5), J6.5 (Pin_5), J7.6 (Pin_6), J8.6 (Pin_6)
- net I2C_SCL: now also J10.3 (Pin_3), J11.1 (Pin_1)
- net I2C_SDA: now also J10.2 (Pin_2), J11.2 (Pin_2)
- net PA10: now also J17.3 (Pin_3), J18.2 (Pin_2)
- net PA11: now also J1.A7 (D-), J1.B7 (D-)
- net PA12: now also J1.A6 (D+), J1.B6 (D+)
- net PA15: now also J4.1 (Pin_1)
- net PA8: now also J3.1 (Pin_1)
- net PA9: now also J3.3 (Pin_3)
- net PB0: now also J8.3 (Pin_3)
- net PB1: now also J8.5 (Pin_5)
- net PB10: now also J17.4 (Pin_4), J18.1 (Pin_1)
- net PB11: now also J13.3 (Pin_3), J16.1 (Pin_1)
- net PB14: now also J7.5 (Pin_5)
- net PB15: now also J7.3 (Pin_3)
- net PB2: now also J13.2 (Pin_2), J16.2 (Pin_2)
- net PB3: now also J4.3 (Pin_3)
- net PB4: now also J5.1 (Pin_1)
- net PB5: now also J5.3 (Pin_3)
- net PB6: now also J6.1 (Pin_1)
- net PB7: now also J6.3 (Pin_3)
- net PB8: now also J8.4 (Pin_4)
- net PB9: now also J8.2 (Pin_2)
- net PC6: now also J7.2 (Pin_2)
- net PC7: now also J7.4 (Pin_4)
- net PD3: now also J17.2 (Pin_2), J18.3 (Pin_3)
- net VBUS: now also C4.1, DCDC1.1 (VIN), DCDC1.3 (STBY), J3.2 (Pin_2), J4.2 (Pin_2), J5.2 (Pin_2), J6.2 (Pin_2)
- new net GND1: J19.1 (Pin_1), J21.1 (Pin_1), J22.1 (Pin_1), J25.1 (Pin_1)
- new net VS: J19.2 (Pin_2), J21.2 (Pin_2), J22.2 (Pin_2), J25.2 (Pin_2)
Other:
- moved on the sheet: J2

Commit message: a
Parts:
- added H1, H2, H3, H4: MountingHole, MountingHole:MountingHole_3.2mm_M3, symbol Mechanical:MountingHole
