File: kicad/MDhubv2/Mdhubv2.kicad_pcb (KiCad board)
At the start: 2 copper layers, 45 parts, among them J1 USB_C_Receptacle_USB2.0_14P, J12 Conn_01x04_Pin, J14 Conn_01x02_Pin, J15 Conn_01x02_Pin, J19 Conn_01x02_Pin, J2 Conn_01x04_Pin, J20 Conn_01x04_Pin, J21 Conn_01x02_Pin, J22 Conn_01x02_Pin, J25 Conn_01x02_Pin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

Commit message: a
Parts:
- added H1: MountingHole, MountingHole:MountingHole_3.2mm_M3, F.Cu at (186.7, 101.6)
- added H2: MountingHole, MountingHole:MountingHole_3.2mm_M3, F.Cu at (133.3, 101.6)
- added H3: MountingHole, MountingHole:MountingHole_3.2mm_M3, F.Cu at (186.2, 140.5)
- added H4: MountingHole, MountingHole:MountingHole_3.2mm_M3, F.Cu at (133.1, 126.0)
- moved G*** 15.7 mm to (133.5, 109.6), turned to -90 degrees
- moved G*** 11.2 mm to (129.9, 117.6), turned to -90 degrees
- moved J30 9.40 mm to (186.7, 128.8)
- moved J28 9.40 mm to (186.7, 115.1)
- moved J29 9.40 mm to (186.7, 121.9)
- moved G*** 6.65 mm to (133.4, 117.7), turned to -90 degrees
Routing:
- net GND: track 60.7 -> 47.0 mm
- net ADC1: track 40.6 -> 49.9 mm
- net ADC0: track 46.2 -> 55.6 mm
- net +3V3: track 186.5 -> 178.8 mm
- net ADC2: track 48.6 -> 55.7 mm
Other:
- board outline added: 91.9 x 47.2 mm

Commit message: a
Routing:
- net CAN_H: track 27.9 -> 31.5 mm
- net ADC1: track 49.9 -> 46.8 mm
- net +3V3: track 178.8 -> 181.5 mm
- net CAN_H2: track 56.5 -> 55.1 mm
- net CAN_L2: track 69.0 -> 67.9 mm
- net PC6: track 44.2 -> 43.1 mm
- net ADC0: track 55.6 -> 54.5 mm
- net ADC3: track 33.8 -> 32.9 mm
- net VBUS: track 132.4 -> 133.2 mm
- net ADC2: track 55.7 -> 54.8 mm
- net PB14: track 35.0 -> 34.3 mm
- net PC7: track 42.0 -> 41.4 mm
- net CAN_L: track 25.3 -> 24.7 mm
- net PB9: track 23.7 -> 23.2 mm
