File: kicad/MD_mini/MD_mini.kicad_pcb (KiCad board)
At the start: 2 copper layers, 74.9 x 31.8 mm, 46 parts, among them J1 Conn_01x02_Pin, J2 Conn_01x06_Pin, J3 Conn_01x02_Pin, J4 Conn_01x02_Pin, U1 IRS2003, U2 SCM3723ASA, U3 IRS2003, U7 IRS2003, U8 IRS2003, U9 SCM3723ASA

Commit message: a
Parts:
- added H1: MountingHole, MountingHole:MountingHole_3.2mm_M3, F.Cu at (107.9, 101.4)
- added H2: MountingHole, MountingHole:MountingHole_3.2mm_M3, F.Cu at (107.9, 109.4)
- added H3: MountingHole, MountingHole:MountingHole_3.2mm_M3, F.Cu at (118.9, 94.0)
- added H4: MountingHole, MountingHole:MountingHole_3.2mm_M3, F.Cu at (114.3, 127.3)
- C1, C2, C3, C4, C6, C7, C8, Q1, Q2, Q3, Q4, Q5, Q6, Q7, Q8: moved to B.Cu
- U2, U9: moved to F.Cu
- moved U2 19.8 mm to (184.8, 114.9), turned to 180 degrees
- moved J1 18.3 mm to (160.6, 113.2)
- moved C6 15.6 mm to (185.1, 100.3)
- moved C2 15.5 mm to (185.2, 107.6)
- moved D8 15.3 mm to (147.9, 121.9), turned to 180 degrees
- moved D7 14.9 mm to (147.9, 123.9)
- moved R8 13.6 mm to (182.6, 100.3), turned to 180 degrees
- moved R9 13.6 mm to (182.6, 102.9), turned to 180 degrees
- moved D5 13.6 mm to (147.9, 107.1), turned to 180 degrees
- moved D3 13.6 mm to (182.6, 98.6)
- moved R1 13.6 mm to (182.6, 110.1)
- moved D1 13.6 mm to (182.6, 105.7)
- moved R2 13.6 mm to (182.6, 107.6), turned to 180 degrees
- moved U1 12.2 mm to (189.7, 108.2)
- moved U8 12.2 mm to (189.7, 101.0)
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Connections:
- D7 pad 2: ch2_1 -> ch2_2
- D8 pad 1: ch2_1 -> ch2_2
- J1 pad 1: VCC -> GND
- J1 pad 2: GND -> VCC
- J3 pad 1: ch2_2 -> ch2_1
- J3 pad 2: ch2_1 -> ch2_2
- R14 pad 1: ch2_2 -> ch2_1
Routing:
- net GND: track 0.00 -> 73.6 mm, vias 0 -> 53
- net VCC: track 0.00 -> 66.6 mm, vias 0 -> 59
- net Net-(U2-OUTA): track 0.00 -> 32.7 mm, vias 0 -> 1
- net ch1_2: track 0.00 -> 25.0 mm, vias 0 -> 59
- net ch2_1: track 0.00 -> 24.6 mm, vias 0 -> 59
- net ch1_1: track 0.00 -> 21.7 mm, vias 0 -> 59
- net Net-(Q4-G): track 0.00 -> 21.5 mm
- net ch2_2: track 0.00 -> 21.1 mm, vias 0 -> 59
- net Net-(Q2-G): track 0.00 -> 20.4 mm
- net Net-(Q7-G): track 0.00 -> 19.7 mm
- net Net-(Q6-G): track 0.00 -> 18.9 mm
- net Net-(J2-Pin_6): track 0.00 -> 17.8 mm
- net Net-(U8-HIN): track 0.00 -> 16.1 mm, vias 0 -> 1
- net Net-(J2-Pin_1): track 0.00 -> 13.5 mm
- net Net-(U2-OUTB): track 0.00 -> 12.7 mm, vias 0 -> 1
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- added copper zone on B.Cu, net GND
- added copper zone on F.Cu, net GND
- added copper zone on B.Cu, net VCC
- added copper zone on F.Cu, net VCC
- added copper zone on B.Cu, net ch1_1
- added copper zone on F.Cu, net ch1_1
- added copper zone on B.Cu, net ch1_2
- added copper zone on F.Cu, net ch1_2
- added copper zone on B.Cu, net ch2_1
- added copper zone on F.Cu, net ch2_1
- added copper zone on B.Cu, net ch2_2
- added copper zone on F.Cu, net ch2_2
Other:
- board size 74.9 x 31.8 mm -> 58.6 x 36.3 mm

Commit message: a
Parts:
- removed J2: Conn_01x06_Pin, Connector_PinHeader_2.54mm:PinHeader_1x06_P2.54mm_Horizontal
- added J6: Conn_02x03_Odd_Even, Connector_PinHeader_2.54mm:PinHeader_2x03_P2.54mm_Horizontal, F.Cu at (195.1, 115.3)
- U2: moved to B.Cu
- moved U9 8.51 mm to (183.9, 114.8)
- moved C3 6.58 mm to (200.7, 114.3)
- moved U7 6.10 mm to (189.5, 121.9)
- moved C8 6.10 mm to (185.0, 121.3)
- moved R11 5.59 mm to (182.6, 120.8)
- moved D4 5.59 mm to (182.6, 119.0)
- moved R12 5.59 mm to (182.6, 123.3)
- moved C4 1.65 mm to (185.2, 126.9)
- moved R5 1.65 mm to (182.6, 126.9)
- moved R6 1.65 mm to (182.6, 129.4)
- moved C5 1.65 mm to (194.4, 124.6)
- moved D2 1.65 mm to (182.6, 125.1)
- moved U3 1.65 mm to (189.7, 127.5)
- moved U2 0.18 mm to (184.9, 114.8)
Connections:
- net Net-(J2-Pin_1) renamed VDD
- net Net-(J2-Pin_6) renamed GND1
Routing:
- net GND: track 73.6 -> 36.7 mm, vias 53 -> 51
- net VCC: track 66.6 -> 32.7 mm, vias 59 -> 58
- net ch2_2: track 21.1 -> 5.88 mm, vias 59 -> 58
- net ch1_2: track 25.0 -> 13.9 mm, vias 59 -> 58
- net Net-(U2-OUTA): track 32.7 -> 22.2 mm, vias 1 -> 0
- net Net-(U1-HIN): track 10.5 -> 17.8 mm
- net Net-(Q6-G): track 18.9 -> 11.9 mm
- net Net-(U8-HIN): track 16.1 -> 22.8 mm
- net Net-(Q3-G): track 5.39 -> 0.71 mm
- net Net-(J6-Pin_2): track 5.32 -> 9.95 mm
- net VDD: track 13.5 -> 18.0 mm
- net GND1: track 17.8 -> 13.6 mm
- net Net-(D2-K): track 4.16 -> 0.00 mm
- net Net-(U3-LO): track 3.72 -> 0.00 mm
- net Net-(U3-HO): track 3.72 -> 0.00 mm
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
Commit message: a
Parts:
- moved C3 8.24 mm to (195.5, 120.8), turned to -90 degrees
- moved C8 1.52 mm to (186.6, 121.3)
- moved D4 1.52 mm to (184.2, 119.0)
- moved R11 1.52 mm to (184.2, 120.8)
- moved R12 1.52 mm to (184.2, 123.3)
- moved U7 1.52 mm to (191.0, 121.9)
- moved D2 1.35 mm to (184.0, 125.3)
- moved U3 1.35 mm to (191.1, 127.7)
- moved C4 1.35 mm to (186.5, 127.0)
- moved R5 1.35 mm to (184.0, 127.0)
- moved R6 1.35 mm to (184.0, 129.6)
- moved C5 1.29 mm to (195.6, 125.0)
- moved U2 0.56 mm to (185.5, 114.8)
Routing:
- net VCC: track 32.7 -> 65.5 mm, vias 58 -> 85
- net GND: track 36.7 -> 59.5 mm, vias 51 -> 53
- net ch2_2: track 5.88 -> 21.3 mm, vias 58 -> 59
- net Net-(Q6-G): track 11.9 -> 26.4 mm
- net ch1_2: track 13.9 -> 24.7 mm, vias 58 -> 59
- net Net-(Q3-G): track 0.71 -> 7.55 mm
- net Net-(Q5-G): track 4.25 -> 10.5 mm
- net Net-(U2-OUTA): track 22.2 -> 28.1 mm
- net Net-(Q4-G): track 19.1 -> 24.8 mm
- net Net-(D2-K): track 0.00 -> 4.16 mm
- net Net-(U3-LO): track 0.00 -> 3.72 mm
- net Net-(U3-HO): track 0.00 -> 3.72 mm
- net VDD: track 18.0 -> 14.3 mm, vias 0 -> 1
- net Net-(U1-HIN): track 17.8 -> 16.0 mm
- net ch2_1: track 23.3 -> 24.8 mm
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
Commit message: a
Parts:
- added J2: Conn_01x03_Pin, Connector_PinHeader_2.54mm:PinHeader_1x03_P2.54mm_Vertical, F.Cu at (143.4, 96.5)
- added U4: ACS711xEXLT-15AB, Sensor_Current:Allegro_QFN-12-10-1EP_3x3mm_P0.5mm, B.Cu at (170.2, 113.5)
- moved H3 23.8 mm to (119.9, 117.9)
- moved U9 0.55 mm to (184.4, 114.8)
- moved Q5 0.46 mm to (174.2, 118.8)
- moved Q6 0.46 mm to (162.5, 118.8)
Connections:
- J1 pad 2: VCC -> Net-(J1-Pin_2)
Routing:
- net Net-(J2-Pin_1): track 0.00 -> 45.7 mm, vias 0 -> 1
- net Net-(J2-Pin_3): track 0.00 -> 41.0 mm, vias 0 -> 1
- net Net-(J2-Pin_2): track 0.00 -> 40.6 mm, vias 0 -> 1
- net Net-(Q6-G): track 26.4 -> 37.9 mm
- net ch2_1: track 24.8 -> 20.9 mm, vias 59 -> 58
- net ch1_2: track 24.7 -> 22.3 mm, vias 59 -> 47
- net VCC: track 65.5 -> 66.8 mm, vias 85 -> 75
- net ch2_2: track 21.3 -> 22.0 mm
- net Net-(U8-HIN): track 21.7 -> 21.1 mm
- net Net-(Q4-G): track 24.8 -> 24.7 mm, vias 0 -> 2
- net Net-(J1-Pin_2): vias 0 -> 5
- added copper zone on B.Cu, net Net-(J1-Pin_2)
- added copper zone on F.Cu, net Net-(J1-Pin_2)

Commit message: a
Parts:
- removed H1, H2, H3, H4: MountingHole, MountingHole:MountingHole_3.2mm_M3

Commit message: a
Parts:
- added U5: ~, jisaku:SOT-89-3, F.Cu at (186.7, 120.0)
Connections:
- U2 pad 8: VCC -> Net-(U2-VCC2)
- U9 pad 8: VCC -> Net-(U2-VCC2)
Routing:
- net Net-(U2-VCC2): track 0.00 -> 10.8 mm, vias 0 -> 1
- net GND: track 59.5 -> 64.4 mm, vias 53 -> 54
- net ch2_1: track 20.9 -> 24.5 mm
- net VCC: track 66.8 -> 63.7 mm
- net VDD: track 14.3 -> 13.8 mm
- net Net-(J6-Pin_3): track 6.88 -> 6.37 mm
Other:
- board text added: "GND"
- board text added: "Vcc"

Commit message: a
Parts:
- moved Q6 1.38 mm to (161.1, 118.8), turned to 90 degrees
- moved Q7 1.26 mm to (161.2, 101.3), turned to 90 degrees
- moved Q2 1.25 mm to (161.2, 108.2), turned to 90 degrees
- moved Q5 1.02 mm to (173.2, 118.8), turned to 90 degrees
- moved Q8 1.01 mm to (173.2, 101.3), turned to 90 degrees
- moved Q1 1.00 mm to (173.2, 108.2), turned to 90 degrees
- moved Q4 0.87 mm to (161.6, 127.0), turned to 90 degrees
- moved Q3 0.55 mm to (173.8, 126.6), turned to 90 degrees
Routing:
- net Net-(Q6-G): track 37.9 -> 26.0 mm, vias 0 -> 2
- net Net-(Q8-G): track 5.64 -> 14.5 mm, vias 0 -> 2
- net Net-(Q1-G): track 6.54 -> 15.3 mm, vias 0 -> 2
- net Net-(Q3-G): track 7.55 -> 14.1 mm
- net Net-(Q7-G): track 19.7 -> 26.0 mm, vias 0 -> 2
- net Net-(Q5-G): track 10.9 -> 16.4 mm, vias 0 -> 2
- net Net-(Q2-G): track 20.4 -> 25.5 mm, vias 0 -> 2
- net Net-(Q4-G): track 24.7 -> 28.6 mm
- net ch1_2: track 22.3 -> 26.2 mm, vias 47 -> 43
- net ch1_1: track 21.7 -> 20.3 mm, vias 59 -> 49
- net ch2_1: track 24.5 -> 25.4 mm, vias 58 -> 47
- net VCC: vias 75 -> 54
- net ch2_2: vias 59 -> 47
- net Net-(J1-Pin_2): vias 5 -> 13
- net GND: vias 54 -> 53

Commit message: test
Routing:
- net ch1_2: track 26.2 -> 27.3 mm
- net Net-(Q7-G): track 26.0 -> 25.1 mm
- net ch2_1: track 25.4 -> 24.7 mm
- net Net-(Q2-G): track 25.5 -> 26.1 mm
- net VCC: track 63.7 -> 63.9 mm, vias 54 -> 49
