File: kicad/MD_mini/MD_mini.kicad_pcb (KiCad board)
At the start: 2 copper layers, 58.6 x 36.3 mm, 51 parts, among them J1 Conn_01x02_Pin, J2 Conn_01x03_Pin, J3 Conn_01x02_Pin, J4 Conn_01x02_Pin, J6 Conn_02x03_Odd_Even, U1 IRS2003, U2 SCM3723ASA, U3 IRS2003, U4 ACS711xEXLT-15AB, U7 IRS2003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

Commit message: a
Parts:
- D1, D2, D3, D4: footprint Diode_SMD:D_SOD-323F -> Diode_SMD:D_MicroSMP_AK
- moved D4 0.51 mm to (183.6, 119.0)
- moved D2 0.43 mm to (183.5, 125.3)
- moved D3 0.42 mm to (182.2, 98.7)
- moved D1 0.35 mm to (182.3, 105.7)
Routing:
- net Net-(J2-Pin_3): track 40.7 -> 36.3 mm
- net Net-(D1-K): track 4.21 -> 5.36 mm
- net Net-(J2-Pin_2): track 40.9 -> 40.1 mm

Commit message: a
Parts:
- added D10: LED, LED_SMD:LED_0603_1608Metric_Pad1.05x0.95mm_HandSolder, B.Cu at (192.3, 112.7)
- added D9: LED, LED_SMD:LED_0603_1608Metric_Pad1.05x0.95mm_HandSolder, B.Cu at (194.7, 97.4)
- added R10: 10, Resistor_SMD:R_0603_1608Metric_Pad0.98x0.95mm_HandSolder, B.Cu at (182.8, 108.8)
- added R15: 10, Resistor_SMD:R_0603_1608Metric_Pad0.98x0.95mm_HandSolder, B.Cu at (156.8, 127.0)
- added R16: 10, Resistor_SMD:R_0603_1608Metric_Pad0.98x0.95mm_HandSolder, B.Cu at (183.9, 128.4)
- added R17: 10, Resistor_SMD:R_0603_1608Metric_Pad0.98x0.95mm_HandSolder, B.Cu at (184.1, 122.1)
- added R18: 10, Resistor_SMD:R_0603_1608Metric_Pad0.98x0.95mm_HandSolder, B.Cu at (160.6, 123.0)
- added R19: R, Resistor_SMD:R_0603_1608Metric_Pad0.98x0.95mm_HandSolder, B.Cu at (194.7, 111.8)
- added R20: R, Resistor_SMD:R_0603_1608Metric_Pad0.98x0.95mm_HandSolder, B.Cu at (194.8, 95.9)
- added R3: 10, Resistor_SMD:R_0603_1608Metric_Pad0.98x0.95mm_HandSolder, B.Cu at (156.3, 102.7)
- added R4: 10, Resistor_SMD:R_0603_1608Metric_Pad0.98x0.95mm_HandSolder, B.Cu at (182.7, 101.8)
- added R7: 10, Resistor_SMD:R_0603_1608Metric_Pad0.98x0.95mm_HandSolder, B.Cu at (156.4, 109.6)
- moved C11 6.56 mm to (180.6, 121.1), turned to 0 degrees
- moved C12 5.71 mm to (181.4, 118.8)
- moved U5 3.32 mm to (182.8, 120.0), turned to 90 degrees
- moved C9 1.40 mm to (189.5, 104.0)
- moved C10 1.37 mm to (178.6, 104.0)
- moved R9 1.05 mm to (182.7, 103.9)
- moved C7 0.47 mm to (195.0, 99.0), turned to 0 degrees
- moved R6 0.30 mm to (183.9, 129.9)
- moved R2 0.26 mm to (182.8, 107.3)
- moved R12 0.26 mm to (184.1, 123.6)
- moved R1 0.24 mm to (182.8, 110.3)
- moved R5 0.18 mm to (184.0, 126.9)
- moved R11 0.18 mm to (184.1, 120.6)
- moved D2 0.08 mm to (183.5, 125.2)
- moved R8 0.08 mm to (182.7, 100.3)
Connections:
- J6 pad 1: VDD -> Net-(J6-Pin_1)
- J6 pad 2: Net-(J6-Pin_2) -> VDD
- J6 pad 5: Net-(J6-Pin_5) -> GND1
- J6 pad 6: GND1 -> Net-(J6-Pin_6)
- U2 pad 2: Net-(J6-Pin_2) -> Net-(J6-Pin_1)
- U2 pad 3: Net-(J6-Pin_4) -> Net-(J6-Pin_3)
- U9 pad 2: Net-(J6-Pin_5) -> Net-(J6-Pin_6)
- U9 pad 3: Net-(J6-Pin_3) -> Net-(J6-Pin_4)
Routing:
- net Net-(J6-Pin_2): track 9.99 -> 0.00 mm
- net Net-(J6-Pin_1): track 0.00 -> 8.98 mm
- net Net-(D10-A): track 12.5 -> 20.4 mm, vias 1 -> 3
- net VCC: track 65.8 -> 59.6 mm, vias 80 -> 79
- net GND1: track 12.4 -> 6.88 mm
- net Net-(U8-HIN): track 21.2 -> 26.2 mm, vias 1 -> 3
- net GND: track 67.9 -> 72.1 mm
- net Net-(J6-Pin_6): track 0.00 -> 4.07 mm
- net Net-(J6-Pin_5): track 3.67 -> 0.00 mm
- net Net-(Q2-G): track 32.1 -> 35.5 mm
- net Net-(J6-Pin_3): track 6.34 -> 9.04 mm
- net ch2_2: track 24.2 -> 26.2 mm
- net ch1_2: track 27.7 -> 29.7 mm
- net Net-(J6-Pin_4): track 5.59 -> 7.53 mm
- net Net-(Q1-G): track 17.3 -> 19.1 mm
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
Commit message: a
Parts:
- added G***: LOGO, _gazou:drive, F.Cu at (157.5, 101.5)
- added G***: LOGO, _gazou:blackpulsedrive, F.Cu at (157.7, 104.2)

Commit message: a
Changed lines of the file:
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@@
 	)
 	(segment
-		(start 173.27 129.032)
+		(start 173.0414 128.8034)
 		(end 171.873 127.635)
 		(width 0.2)
@@
 	)
 	(segment
-		(start 182.084 129.032)
-		(end 173.27 129.032)
-		(width 0.2)
-		(layer "F.Cu")
-		(net 5)
-	)
-	(segment
-		(start 182.3126 128.8034)
-		(end 182.084 129.032)
-		(width 0.2)
-		(layer "F.Cu")
-		(net 5)
-	)
-	(segment
 		(start 186.69 128.8034)
-		(end 182.3126 128.8034)
+		(end 173.0414 128.8034)
 		(width 0.2)
 		(layer "F.Cu")
@@
 	)
 	(segment
-		(start 181.6682 123.7234)
-		(end 181.987165 124.042365)
+		(start 173.840665 122.845765)
+		(end 172.490065 122.845765)
 		(width 0.2)
 		(layer "F.Cu")
@@
 	)
 	(segment
-		(start 173.840665 122.845765)
-		(end 174.7183 123.7234)
+		(start 175.037265 124.042365)
+		(end 173.840665 122.845765)
 		(width 0.2)
 		(layer "F.Cu")
@@
 	)
 	(segment
-		(start 172.490065 122.845765)
-		(end 173.840665 122.845765)
-		(width 0.2)
-		(layer "F.Cu")
-		(net 17)
-	)
-	(segment
-		(start 174.7183 123.7234)
-		(end 181.6682 123.7234)
-		(width 0.2)
-		(layer "F.Cu")
+		(start 181.987165 124.042365)
+		(end 175.037265 124.042365)
+		(width 0.2)
+		(layer "F.Cu")

Commit message: a
Parts:
- added U6: ACS711xEXLT-15AB, Sensor_Current:Allegro_QFN-12-10-1EP_3x3mm_P0.5mm, B.Cu at (154.7, 115.8)
- J2: value Conn_01x03_Pin -> Conn_01x04_Pin; footprint Connector_PinHeader_2.54mm:PinHeader_1x03_P2.54mm_Vertical -> Connector_PinHeader_2.54mm:PinHeader_1x04_P2.54mm_Vertical
- J3, J4: footprint Connector_AMASS:AMASS_XT30PW-M_1x02_P2.50mm_Horizontal -> Connector_AMASS:AMASS_XT30PW-F_1x02_P2.50mm_Horizontal
- R3, R4: value 10 -> 10k
- moved J2 19.5 mm to (152.0, 113.9), turned to -90 degrees
- moved U4 15.6 mm to (154.7, 111.5), turned to 180 degrees
- moved J3 7.59 mm to (151.1, 125.3)
- moved Q3 4.94 mm to (168.9, 126.9)
- moved R18 4.72 mm to (158.3, 118.9)
- moved J4 4.37 mm to (151.1, 107.4)
- moved R14 4.18 mm to (147.1, 123.5), turned to 180 degrees
- moved D5 3.99 mm to (147.3, 103.2)
- moved D6 3.99 mm to (147.3, 104.8)
- moved Q4 3.84 mm to (157.8, 126.8)
- moved R20 3.37 mm to (195.5, 99.2)
- moved C7 3.37 mm to (195.6, 102.3)
- moved D9 3.37 mm to (195.4, 100.7)
- moved R3 2.70 mm to (158.6, 101.3), turned to 0 degrees
- moved R7 2.66 mm to (158.6, 108.2), turned to 0 degrees
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Connections:
- net Net-(J2-Pin_2) renamed cur_1
- D5 pad 1: ch1_2 -> ch1_1
- D6 pad 2: ch1_2 -> ch1_1
- D7 pad 2: ch2_2 -> ch2_1
- D8 pad 1: ch2_2 -> ch2_1
- J1 pad 2: Net-(J1-Pin_2) -> VCC
- J2 pad 1: Net-(J2-Pin_1) -> VDDA
- J2 pad 3: Net-(J2-Pin_3) -> cur_2
- J3 pad 1: ch2_1 -> ch2_2
- J3 pad 2: ch2_2 -> ch2_1
- J4 pad 1: ch1_1 -> ch1_2
- J4 pad 2: ch1_2 -> ch1_1
- Q2 pad 3: GND -> Net-(Q2-S)
- Q4 pad 3: GND -> Net-(Q4-S)
- Q6 pad 3: GND -> Net-(Q4-S)
- Q7 pad 3: GND -> Net-(Q2-S)
- R13 pad 1: ch1_1 -> ch1_2
- R14 pad 1: ch2_1 -> ch2_2
- R15 pad 1: GND -> Net-(Q4-S)
- R18 pad 1: GND -> Net-(Q4-S)
- R3 pad 1: GND -> Net-(Q2-S)
- R7 pad 1: GND -> Net-(Q2-S)
- U4 pad 1: Net-(J1-Pin_2) -> Net-(Q2-S)
- U4 pad 10: Net-(J2-Pin_3) -> VDDA
- U4 pad 2: VCC -> GND
- U4 pad 3: Net-(J2-Pin_1) -> GNDS
Routing:
- net Net-(J2-Pin_1): track 45.8 -> 0.00 mm, vias 1 -> 0
- net Net-(J2-Pin_3): track 36.3 -> 0.00 mm, vias 1 -> 0
- net cur_1: track 40.1 -> 6.41 mm, vias 1 -> 0
- net Net-(Q2-G): track 35.5 -> 2.59 mm, vias 2 -> 0
- net GNDS: track 0.00 -> 23.9 mm, vias 0 -> 1
- net Net-(Q7-G): track 26.2 -> 2.92 mm, vias 2 -> 0
- net ch1_2: track 29.7 -> 7.32 mm, vias 43 -> 1
- net Net-(Q1-G): track 19.1 -> 0.00 mm, vias 2 -> 0
- net GND: track 72.1 -> 89.1 mm, vias 53 -> 4
- net Net-(D10-A): track 20.4 -> 3.89 mm, vias 3 -> 0
- net Net-(Q8-G): track 16.1 -> 0.00 mm, vias 2 -> 0
- net ch1_1: track 22.6 -> 8.90 mm, vias 49 -> 1
- net VCC: track 59.6 -> 46.5 mm, vias 79 -> 4
- net cur_2: track 0.00 -> 10.7 mm, vias 0 -> 2
- net VDDA: track 0.00 -> 9.60 mm, vias 0 -> 2
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- added copper zone on B.Cu, net Net-(Q2-S)
- added copper zone on B.Cu, net Net-(Q4-S)
- removed copper zone on F.Cu, net GND
- removed copper zone on B.Cu, net Net-(J1-Pin_2)
- removed copper zone on F.Cu, net Net-(J1-Pin_2)
Other:
- board size 58.6 x 36.3 mm -> 60.6 x 32.3 mm
- board text removed: "GND"
- board text removed: "Vcc"

Commit message: a
Parts:
- added C13: 0.1u, Capacitor_SMD:C_0603_1608Metric, B.Cu at (181.0, 116.1)
- added C14: 0.1u, Capacitor_SMD:C_0603_1608Metric, B.Cu at (181.0, 113.1)
- added C15: C, Capacitor_SMD:C_0603_1608Metric, B.Cu at (221.7, 125.3)
- added C16: C, Capacitor_SMD:C_0603_1608Metric, B.Cu at (221.7, 122.7)
- added C17: C, Capacitor_SMD:C_0603_1608Metric, B.Cu at (166.2, 122.9)
- added C18: C, Capacitor_SMD:C_0603_1608Metric, B.Cu at (159.7, 123.0)
- added C19: C, Capacitor_SMD:C_0603_1608Metric, B.Cu at (222.1, 115.4)
- added C20: C, Capacitor_SMD:C_0603_1608Metric, B.Cu at (221.7, 112.7)
- added C21: C, Capacitor_SMD:C_0603_1608Metric, B.Cu at (221.7, 110.2)
- added C22: C, Capacitor_SMD:C_0603_1608Metric, B.Cu at (221.7, 107.7)
- added R21: R, Resistor_SMD:R_0603_1608Metric_Pad0.98x0.95mm_HandSolder, B.Cu at (225.9, 125.3)
- added R22: R, Resistor_SMD:R_0603_1608Metric_Pad0.98x0.95mm_HandSolder, B.Cu at (225.9, 122.7)
- added R23: R, Resistor_SMD:R_0603_1608Metric_Pad0.98x0.95mm_HandSolder, B.Cu at (170.8, 122.9)
- added R24: R, Resistor_SMD:R_0603_1608Metric_Pad0.98x0.95mm_HandSolder, B.Cu at (162.8, 123.0)
- added R25: R, Resistor_SMD:R_0603_1608Metric_Pad0.98x0.95mm_HandSolder, B.Cu at (225.9, 115.2)
- added R26: R, Resistor_SMD:R_0603_1608Metric_Pad0.98x0.95mm_HandSolder, B.Cu at (225.9, 112.7)
- added R27: R, Resistor_SMD:R_0603_1608Metric_Pad0.98x0.95mm_HandSolder, B.Cu at (225.9, 110.2)
- added R28: R, Resistor_SMD:R_0603_1608Metric_Pad0.98x0.95mm_HandSolder, B.Cu at (225.9, 107.7)
- moved C11 1.18 mm to (181.4, 122.0), turned to 90 degrees
- moved D3 0.20 mm to (182.2, 99.2)
Routing:
- net GND: track 89.1 -> 38.1 mm, vias 4 -> 132
- net Net-(Q2-G): track 2.59 -> 33.1 mm, vias 0 -> 2
- net Net-(Q7-G): track 2.92 -> 26.3 mm, vias 0 -> 2
- net Net-(Q1-G): track 0.00 -> 17.5 mm, vias 0 -> 2
- net Net-(D10-A): track 3.89 -> 21.3 mm, vias 0 -> 3
- net Net-(Q8-G): track 0.00 -> 17.0 mm, vias 0 -> 2
- net ch1_2: track 7.32 -> 22.9 mm, vias 1 -> 55
- net ch1_1: track 8.90 -> 24.2 mm, vias 1 -> 56
- net VDD: track 9.58 -> 15.3 mm, vias 0 -> 1
- net VCC: track 46.5 -> 41.3 mm, vias 4 -> 125
- net Net-(C17-Pad2): track 0.00 -> 3.50 mm
- net ch2_2: track 24.9 -> 28.4 mm, vias 3 -> 49
- net Net-(U2-OUTA): track 28.5 -> 31.2 mm
- net Net-(Q4-S): track 2.66 -> 4.95 mm, vias 0 -> 12
- net ch2_1: track 26.6 -> 28.8 mm, vias 3 -> 45
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- added copper zone on F.Cu, net GND
- added copper zone on F.Cu, net Net-(Q2-S)
- added copper zone on F.Cu, net Net-(Q4-S)
Other:
- board size 60.6 x 32.3 mm -> 60.6 x 31.8 mm
- board text added: "104"
- board text added: "470"
