File: kicad/MD_mini/MD_mini_v2.kicad_sch (KiCad schematic)
At the start: 89 parts, among them J1 Conn_01x02_Pin, J2 Conn_02x05_Odd_Even, J3 Conn_01x02_Pin, J4 Conn_01x02_Pin, J5 Conn_01x05_Pin, J6 Conn_01x05_Pin, J7 Conn_01x04_Pin, J8 Conn_01x04_Pin, U1 IRS2003, U10 BD4104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

Commit message: a
Changed lines of the file:
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@@
 	(paper "A4")
 	(junction
+		(at 86.36 52.07)
+		(diameter 0)
+		(color 0 0 0 0)
+	)
+	(junction
 		(at 115.57 31.75)
 		(diameter 0)
@@
 	)
 	(junction
-		(at 86.36 49.53)
-		(diameter 0)
-		(color 0 0 0 0)
-	)
-	(junction
 		(at 236.22 48.26)
 		(diameter 0)
@@
 	(wire
 		(pts
-			(xy 176.53 92.71) (xy 176.53 90.17)
-		)
-		(stroke
-			(width 0)
-			(type default)
-		)
-	)
-	(wire
-		(pts
 			(xy 106.68 83.82) (xy 115.57 83.82)
 		)
@@
 	(wire
 		(pts
-			(xy 176.53 90.17) (xy 189.23 90.17)
-		)
-		(stroke
-			(width 0)
-			(type default)
-		)
-	)
-	(wire
-		(pts
 			(xy 242.57 95.25) (xy 242.57 92.71)
 		)
@@
 	(wire
 		(pts
-			(xy 77.47 52.07) (xy 77.47 48.26)
-		)
-		(stroke
-			(width 0)
-			(type default)
-		)
-	)
-	(wire
-		(pts
 			(xy 67.31 121.92) (xy 78.74 121.92)
 		)
@@
 	(wire
 		(pts
+			(xy 177.8 90.17) (xy 189.23 90.17)
+		)
+		(stroke
+			(width 0)
+			(type default)
+		)
+	)
+	(wire
+		(pts
 			(xy 193.04 77.47) (xy 201.93 77.47)
 		)
@@
 	(wire
 		(pts
-			(xy 86.36 48.26) (xy 86.36 49.53)
-		)
-		(stroke
-			(width 0)
-			(type default)
-		)
-	)
-	(wire
-		(pts
 			(xy 43.18 106.68) (xy 43.18 110.49)
 		)
@@
 	(wire
 		(pts
-			(xy 77.47 48.26) (xy 86.36 48.26)
-		)
-		(stroke
-			(width 0)
-			(type default)
-		)
-	)
-	(wire
-		(pts
 			(xy 35.56 39.37) (xy 49.53 39.37)
 		)
@@
 	(wire
 		(pts
-			(xy 176.53 92.71) (xy 177.8 92.71)
-		)
-		(stroke
-			(width 0)
-			(type default)
-		)
-	)
-	(wire
-		(pts
 			(xy 25.4 127) (xy 25.4 121.92)
 		)
@@
 	(wire
 		(pts
-			(xy 49.53 52.07) (xy 77.47 52.07)
+			(xy 49.53 52.07) (xy 86.36 52.07)
 		)
 		(stroke
@@
 	(wire
 		(pts
-			(xy 177.8 92.71) (xy 177.8 52.07)
-		)
-		(stroke
+			(xy 177.8 90.17) (xy 177.8 52.07)
+		)
+		(stroke
