File: kicad/MD_mini/MD_mini_v2.kicad_sch (KiCad schematic)
At the start: 89 parts, among them J1 Conn_01x02_Pin, J2 Conn_02x05_Odd_Even, J3 Conn_01x02_Pin, J4 Conn_01x02_Pin, J5 Conn_01x05_Pin, J6 Conn_01x05_Pin, J7 Conn_01x04_Pin, J8 Conn_01x04_Pin, U1 IRS2003, U10 BD4104, U11 STM32C092KBT6, U2 SCM3723ASA, U3 IRS2003, U4 ACS711xEXLT-15AB, U6 ACS711xEXLT-15AB, U7 IRS2003, U8 IRS2003, U9 SCM3723ASA

Commit message: a
Parts:
- added TP1, TP2, TP3, TP4, TP5, TP6, TP7, TP8: TestPoint, symbol Connector:TestPoint
- R10, R15, R16, R17, R18: value 10 -> 10k
- R7: value 10 -> 01k
Connections:
- net CAN_H: no longer J2.3 (Pin_3)
- net CAN_L: no longer J2.5 (Pin_5)
- net RX: no longer J2.9 (Pin_9)
- net TX: no longer J2.7 (Pin_7)
- net at Q6.1 (G), R12.2, R18.2: now also TP8.1
- net at Q2.1 (G), R1.2, R7.2: now also TP4.1
- net at Q4.1 (G), R15.2, R6.2: now also TP6.1
- net at Q7.1 (G), R3.2, R9.2: now also TP2.1
- net at Q1.1 (G), R10.1, R2.2: now also TP3.1
- net at Q5.1 (G), R11.2, R17.1: now also TP7.1
- net at Q3.1 (G), R16.1, R5.2: now also TP5.1
- net at Q8.1 (G), R4.1, R8.2: now also TP1.1

Commit message: a
Parts:
- removed C15, C16, C17, C18, C19, C20, C21, C22: C, Capacitor_SMD:C_0603_1608Metric, symbol Device:C
- removed R21, R22, R23, R24, R25, R26, R27, R28, R29: R, Resistor_SMD:R_0603_1608Metric_Pad0.98x0.95mm_HandSolder, symbol Device:R
- removed U10: BD4104, jisaku:SOP-J8, symbol jisaku:BD4104
- removed U2, U9: SCM3723ASA, Package_SO:SOIC-8_3.9x4.9mm_P1.27mm, symbol jisaku:SCM3723ASA
- removed U5: ~, jisaku:SOT-89-3, symbol jisaku:NJM78L00SU3
- added C23: 0.1u, Capacitor_SMD:C_0603_1608Metric, symbol Device:C
- added C25: min0.33u, Capacitor_SMD:C_0603_1608Metric, symbol Device:C
- added NJM78L05SU1: ~, jisaku:SOT-89-3, symbol jisaku:NJM78L05SU3
- added NJM78L12SU3, NJM78L33SU1: ~, jisaku:SOT-89-3, symbol jisaku:NJM78L33SU3
- added R43: R, Resistor_SMD:R_0603_1608Metric_Pad0.98x0.95mm_HandSolder, symbol Device:R
- added U2: BD4104, jisaku:SOP-J8, symbol jisaku:BD4104
- added U5: ADuM1201AR, Package_SO:SOIC-8_3.9x4.9mm_P1.27mm, symbol Isolator:ADuM1201AR
- C14: value 0.1u -> min0.33u
Connections:
- net +3V3: no longer J2.2 (Pin_2)
- net +5V: now also C14.1, C25.1, NJM78L05SU1.1 (Vout), NJM78L33SU1.1 (Vout), U5.8 (VDD2); no longer J2.4 (Pin_4)
- net CAN_H: now also J2.3 (Pin_3), R43.2, U2.7 (H)
- net CAN_L: now also J2.5 (Pin_5), R43.1, U2.6 (L)
- net CAN_RX: now also U5.6 (VOB)
- net CAN_TX: now also U5.7 (VIA)
- net GND: now also C24.2, J5.5 (Pin_5), J6.5 (Pin_5), J7.4 (Pin_4), J8.1 (Pin_1), U11.5 (VSS/VSSA), U4.3 (GND), U6.3 (GND), C23.2, C25.2, NJM78L05SU1.2 (GND), NJM78L12SU3.2 (GND), NJM78L33SU1.2 (GND), U5.5 (GND2)
- net GND1: now also U2.2 (GND), U2.8 (STB), U5.4 (GND1); no longer C24.2, J5.5 (Pin_5), J6.5 (Pin_5), J7.4 (Pin_4), J8.1 (Pin_1), U11.5 (VSS/VSSA), U4.3 (GND), U6.3 (GND)
- net PWM1_1: now also U1.2 (HIN), U1.3 (~{LIN})
- net PWM1_2: now also U8.2 (HIN), U8.3 (~{LIN})
- net PWM2_1: now also U3.2 (HIN), U3.3 (~{LIN})
- net PWM2_2: now also U7.2 (HIN), U7.3 (~{LIN})
- net RX: now also J2.9 (Pin_9)
- net TX: now also J2.7 (Pin_7)
- net VCC: now also C12.1, D10.2 (A), NJM78L12SU3.3 (Vin); no longer C1.1, C11.1, C3.1, C5.1, C7.1, D9.2 (A), U1.1 (VCC), U3.1 (VCC), U7.1 (VCC), U8.1 (VCC)
- new net: U2.1 (TX), U5.2 (VOA)
- new net: J2.4 (Pin_4), U2.3 (VCC), U5.1 (VDD1)
- new net: U2.4 (RX), U5.3 (VIB)
- new net: C1.1, C11.1, C13.1, C23.1, C3.1, C5.1, C7.1, D9.2 (A), NJM78L05SU1.3 (Vin), NJM78L12SU3.1 (Vout), NJM78L33SU1.3 (Vin), U1.1 (VCC), U3.1 (VCC), U7.1 (VCC), U8.1 (VCC)
Other:
- moved on the sheet: C12, J2
