File: kicad/MD_mini/MD_mini_v2.kicad_pcb (KiCad board)
At the start: 2 copper layers, 51.2 x 29.8 mm, 84 parts, among them J1 Conn_01x02_Pin, J2 Conn_01x04_Pin, J3 Conn_01x02_Pin, J4 Conn_01x02_Pin, J6 Conn_02x03_Odd_Even, U1 IRS2003, U2 SCM3723ASA, U3 IRS2003, U4 ACS711xEXLT-15AB, U6 ACS711xEXLT-15AB, U7 IRS2003, U8 IRS2003, U9 SCM3723ASA

Commit message: a
Parts:
- removed C10, C9: C, Capacitor_SMD:C_Elec_10x10.2
- removed C11: min0.33u, Capacitor_SMD:C_0603_1608Metric
- removed C12, C13, C14: 0.1u, Capacitor_SMD:C_0603_1608Metric
- removed C15, C16, C17, C18, C19, C20, C21, C22: C, Capacitor_SMD:C_0603_1608Metric
- removed D10, D5, D6, D7, D8: LED, LED_SMD:LED_0603_1608Metric_Pad1.05x0.95mm_HandSolder
- removed J2: Conn_01x04_Pin, Connector_PinHeader_2.54mm:PinHeader_1x04_P2.54mm_Vertical
- removed R13, R14, R19, R21, R22, R23, R24, R25, R26, R27, R28: R, Resistor_SMD:R_0603_1608Metric_Pad0.98x0.95mm_HandSolder
- removed U2, U9: SCM3723ASA, Package_SO:SOIC-8_3.9x4.9mm_P1.27mm
- removed U5: ~, jisaku:SOT-89-3
- C1, C3, C5, C7, D9, R20: moved to F.Cu
- moved R20 36.6 mm to (170.1, 125.5), turned to 180 degrees
- moved D9 35.7 mm to (168.3, 123.9)
- moved C7 29.8 mm to (166.4, 108.5)
- moved C1 28.6 mm to (167.9, 115.6)
- moved C5 22.0 mm to (168.8, 128.5)
- moved C3 21.5 mm to (168.8, 121.5), turned to 90 degrees
Routing:
- net VCC: track 0.00 -> 33.1 mm
- net GNDS: track 0.00 -> 8.45 mm, vias 0 -> 2
- net VDDA: track 0.00 -> 6.41 mm, vias 0 -> 2
- net GND: track 13.4 -> 19.6 mm, vias 1 -> 0
- net Net-(D1-K): track 2.12 -> 3.98 mm
- net Net-(D9-K): track 0.00 -> 1.60 mm
- net Net-(U8-HIN): track 0.00 -> 1.27 mm
- net Net-(U2-OUTB): track 0.00 -> 1.27 mm
- net Net-(U2-OUTA): track 0.00 -> 1.27 mm
- net Net-(U1-HIN): track 0.00 -> 1.27 mm
- net Net-(Q7-G): track 11.8 -> 11.1 mm
- net ch2_1: track 3.94 -> 3.69 mm, vias 0 -> 1
Other:
- board text removed: "104"
- board text removed: "470"

Commit message: a
Changed lines of the file:
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@@
 	)
 	(arc
-		(start 167.784891 119.0752)
+		(start 167.0797 118.7831)
 		(mid 167.403244 118.999285)
-		(end 167.0797 118.7831)
+		(end 167.784891 119.0752)
 		(width 0.2)
 		(layer "F.Cu")
@@
 	)
 	(arc
-		(start 148.714277 104.3689)
+		(start 149.416662 104.077962)
 		(mid 149.094405 104.293287)
-		(end 149.416662 104.077962)
+		(end 148.714277 104.3689)
 		(width 0.889)
 		(layer "B.Cu")
@@
 	)
 	(arc
-		(start 152.5342 101.846278)
+		(start 152.305737 102.397837)
 		(mid 152.474824 102.144779)
-		(end 152.305737 102.397837)
+		(end 152.5342 101.846278)
 		(width 0.889)
 		(layer "B.Cu")
@@
 	)
 	(segment
-		(start 159.865867 127.603832)
-		(end 158.4433 129.0264)
+		(start 158.4433 129.0264)
+		(end 159.865867 127.603832)
 		(width 0.2)
 		(layer "F.Cu")
@@
 	)
 	(arc
-		(start 158.4433 129.19)
+		(start 158.4433 129.0264)
 		(mid 158.409417 129.1082)
-		(end 158.4433 129.0264)
+		(end 158.4433 129.19)
 		(width 0.2)
 		(layer "F.Cu")
@@
 	)
 	(segment
-		(start 160.11245 104.61875)
-		(end 159.91515 104.81605)
+		(start 160.063125 104.668075)
+		(end 160.012025 104.719175)
 		(width 0.2)
 		(layer "F.Cu")
@@
 	)
 	(segment
+		(start 160.161775 104.569425)
+		(end 160.063125 104.668075)
+		(width 0.2)
+		(layer "F.Cu")
+		(net 8)
+	)
+	(segment
+		(start 160.012025 104.719175)
+		(end 159.818275 104.912925)
+		(width 0.2)
+		(layer "F.Cu")
+		(net 8)
+	)
+	(segment
 		(start 159.7214 105.0098)
-		(end 159.91515 104.81605)
+		(end 159.818275 104.912925)
 		(width 0.2)
 		(layer "F.Cu")
@@
 	)
 	(segment
-		(start 160.11245 104.61875)
+		(start 160.161775 104.569425)
 		(end 160.2111 104.5201)
 		(width 0.2)
@@
 	)
 	(arc
-		(start 160.1151 120.0085)
+		(start 160.712617 119.761)
 		(mid 160.389243 119.825323)
-		(end 160.712617 119.761)
+		(end 160.1151 120.0085)
 		(width 0.2)
 		(layer "F.Cu")
@@
 	)
 	(arc
-		(start 159.99135 121.92975)
+		(start 159.743849 121.929749)
 		(mid 159.867599 121.87849)
-		(end 159.743849 121.929749)
+		(end 159.99135 121.92975)
 		(width 0.2)
 		(layer "F.Cu")
@@
 	)
 	(segment
-		(start 156.5675 111.379)
-		(end 156.5675 110.963439)
+		(start 156.5675 110.963439)
+		(end 156.5675 111.171219)
 		(width 0.2)
 		(layer "F.Cu")
@@
 	)
 	(segment
-		(start 156.5675 111.379)
-		(end 156.5675 112.210122)
+		(start 156.5675 111.171219)
+		(end 156.5675 111.58678)
 		(width 0.2)
 		(layer "F.Cu")
@@
 	)
 	(segment
-		(start 156.5675 112.210122)
+		(start 156.5675 111.876383)
+		(end 156.5675 111.58678)
+		(width 0.2)
+		(layer "F.Cu")
+		(net 11)
+	)
+	(segment
+		(start 156.5675 112.543861)
 		(end 156.5675 112.8776)
 		(width 0.2)
@@
 		(start 155.39047 109.370848)
 		(end 156.273653 110.254031)
+		(width 0.2)
+		(layer "F.Cu")
+		(net 11)
+	)
+	(segment
+		(start 156.5675 111.876383)
+		(end 156.5675 112.543861)
 		(width 0.2)
 		(layer "F.Cu")
@@
 	)
 	(segment
+		(start 153.928979 122.773048)
+		(end 152.019 122.773048)
+		(width 0.2)
+		(layer "F.Cu")
+		(net 13)
+	)
+	(segment
+		(start 156.5675 124.958839)
+		(end 156.5675 126.5428)
+		(width 0.2)
+		(layer "F.Cu")
+		(net 13)
+	)
+	(segment
 		(start 154.890918 123.171496)
 		(end 156.48918 124.769758)
@@
 		(net 13)
 	)
-	(segment
-		(start 150.3164 121.8488)
-		(end 150.842199 122.374599)
-		(width 0.2)
-		(layer "F.Cu")
+	(via
+		(at 152.019 122.773048)
+		(size 0.45)
+		(drill 0.3)
+		(layers "F.Cu" "B.Cu")
 		(net 13)
 	)
-	(segment
-		(start 156.5675 124.958839)
-		(end 156.5675 126.5428)
-		(width 0.2)
-		(layer "F.Cu")
-		(net 13)
-	)
-	(segment
-		(start 151.804138 122.773048)
+	(arc
+		(start 154.890918 123.171496)
+		(mid 154.449576 122.876601)
 		(end 153.928979 122.773048)
 		(width 0.2)
 		(layer "F.Cu")
-		(net 13)
-	)
-	(via
-		(at 150.3164 121.8488)
-		(size 0.45)
-		(drill 0.3)
-		(layers "F.Cu" "B.Cu")
 		(net 13)
 	)
@@
 		(net 13)
 	)
-	(arc
-		(start 154.890918 123.171496)
-		(mid 154.449576 122.876601)
-		(end 153.928979 122.773048)
-		(width 0.2)
-		(layer "F.Cu")
+	(segment
+		(start 152.019 122.773048)
+		(end 151.629824 122.773048)
+		(width 0.2)
+		(layer "B.Cu")
 		(net 13)
 	)
-	(arc
-		(start 150.842199 122.374599)
-		(mid 151.28354 122.669494)
-		(end 151.804138 122.773048)
-		(width 0.2)
-		(layer "F.Cu")
+	(segment
+		(start 150.965459 122.497859)
+		(end 150.3164 121.8488)
+		(width 0.2)
+		(layer "B.Cu")
+		(net 13)
+	)
+	(arc
+		(start 150.965459 122.497859)
+		(mid 151.270272 122.701528)
+		(end 151.629824 122.773048)
+		(width 0.2)
+		(layer "B.Cu")
 		(net 13)
 	)
@@
 	)
 	(segment
-		(start 153.084748 101.673248)
-		(end 156.5675 105.156)
+		(start 156.5675 105.156)
+		(end 153.084748 101.673248)
 		(width 0.2)
 		(layer "F.Cu")
@@
 	)
 	(arc
-		(start 159.95698 105.6626)
+		(start 158.995041 106.061048)
 		(mid 159.436382 105.766153)
-		(end 158.995041 106.061048)
+		(end 159.95698 105.6626)
 		(width 0.2)
 		(layer "F.Cu")
@@
 	)
 	(arc
-		(start 161.7296 105.5546)
+		(start 161.468864 105.6626)
 		(mid 161.609973 105.634531)
-		(end 161.468864 105.6626)
-		(width 0.2)
-		(layer "F.Cu")
+		(end 161.7296 105.5546)
+		(width 0.2)
+		(layer "F.Cu")

Commit message: a
Parts:
- removed J6: Conn_02x03_Odd_Even, Connector_PinHeader_2.54mm:PinHeader_2x03_P2.54mm_Horizontal
- added C10: C, Capacitor_SMD:C_Elec_10x10.2, F.Cu at (245.1, 83.2)
- added C11: min0.33u, Capacitor_SMD:C_0603_1608Metric, F.Cu at (263.3, 81.4)
- added C12: 0.1u, Capacitor_SMD:C_0603_1608Metric, F.Cu at (263.3, 83.9)
- added C13: 0.1u, Capacitor_SMD:C_0603_1608Metric, F.Cu at (263.3, 86.4)
- added C14: 0.1u, Capacitor_SMD:C_0603_1608Metric, F.Cu at (263.3, 88.9)
- added C15: C, Capacitor_SMD:C_0603_1608Metric, F.Cu at (267.3, 81.4)
- added C16: C, Capacitor_SMD:C_0603_1608Metric, F.Cu at (267.3, 83.9)
- added C17: C, Capacitor_SMD:C_0603_1608Metric, F.Cu at (267.3, 86.4)
- added C18: C, Capacitor_SMD:C_0603_1608Metric, F.Cu at (267.3, 88.9)
- added C19: C, Capacitor_SMD:C_0603_1608Metric, F.Cu at (271.3, 81.4)
- added C20: C, Capacitor_SMD:C_0603_1608Metric, F.Cu at (271.3, 83.9)
- added C21: C, Capacitor_SMD:C_0603_1608Metric, F.Cu at (271.3, 86.4)
- added C22: C, Capacitor_SMD:C_0603_1608Metric, F.Cu at (271.3, 88.9)
- added C23: C, Capacitor_SMD:C_0603_1608Metric, F.Cu at (267.0, 102.9)
- added C9: C, Capacitor_SMD:C_Elec_10x10.2, F.Cu at (245.1, 71.3)
- added D10: LED, LED_SMD:LED_0603_1608Metric_Pad1.05x0.95mm_HandSolder, F.Cu at (248.3, 100.8)
- added D5: LED, LED_SMD:LED_0603_1608Metric_Pad1.05x0.95mm_HandSolder, F.Cu at (248.3, 90.4)
- added D6: LED, LED_SMD:LED_0603_1608Metric_Pad1.05x0.95mm_HandSolder, F.Cu at (248.3, 93.0)
- added D7: LED, LED_SMD:LED_0603_1608Metric_Pad1.05x0.95mm_HandSolder, F.Cu at (248.3, 95.6)
- added D8: LED, LED_SMD:LED_0603_1608Metric_Pad1.05x0.95mm_HandSolder, F.Cu at (248.3, 98.2)
- added J2: Conn_02x05_Odd_Even, Connector_PinHeader_2.54mm:PinHeader_2x05_P2.54mm_Horizontal, F.Cu at (178.6, 143.9)
- added R13: R, Resistor_SMD:R_0603_1608Metric_Pad0.98x0.95mm_HandSolder, F.Cu at (254.7, 81.4)
- added R14: R, Resistor_SMD:R_0603_1608Metric_Pad0.98x0.95mm_HandSolder, F.Cu at (254.7, 83.9)
- added R19: R, Resistor_SMD:R_0603_1608Metric_Pad0.98x0.95mm_HandSolder, F.Cu at (254.7, 86.4)
- added R21: R, Resistor_SMD:R_0603_1608Metric_Pad0.98x0.95mm_HandSolder, F.Cu at (254.7, 88.9)
- added R22: R, Resistor_SMD:R_0603_1608Metric_Pad0.98x0.95mm_HandSolder, F.Cu at (254.7, 91.4)
- added R23: R, Resistor_SMD:R_0603_1608Metric_Pad0.98x0.95mm_HandSolder, F.Cu at (254.7, 94.0)
- added R24: R, Resistor_SMD:R_0603_1608Metric_Pad0.98x0.95mm_HandSolder, F.Cu at (259.1, 81.4)
- added R25: R, Resistor_SMD:R_0603_1608Metric_Pad0.98x0.95mm_HandSolder, F.Cu at (259.1, 83.9)
- added R26: R, Resistor_SMD:R_0603_1608Metric_Pad0.98x0.95mm_HandSolder, F.Cu at (259.1, 86.4)
- added R27: R, Resistor_SMD:R_0603_1608Metric_Pad0.98x0.95mm_HandSolder, F.Cu at (259.1, 88.9)
- added R28: R, Resistor_SMD:R_0603_1608Metric_Pad0.98x0.95mm_HandSolder, F.Cu at (259.1, 91.4)
- added U10: STM32C011F4Px, Package_SO:TSSOP-20_4.4x6.5mm_P0.65mm, B.Cu at (168.0, 139.0)
- added U2: SCM3723ASA, Package_SO:SOIC-8_3.9x4.9mm_P1.27mm, B.Cu at (165.8, 113.0)
- added U5: ~, jisaku:SOT-89-3, F.Cu at (255.5, 96.0)
- added U9: SCM3723ASA, Package_SO:SOIC-8_3.9x4.9mm_P1.27mm, B.Cu at (165.8, 129.5)
- moved Q8 51.8 mm to (189.6, 134.5), turned to 90 degrees
- moved Q1 45.4 mm to (189.6, 128.1), turned to 90 degrees
- moved Q3 42.9 mm to (189.6, 113.9), turned to 90 degrees
- moved Q5 41.8 mm to (189.6, 120.3), turned to 90 degrees
- moved R9 37.4 mm to (174.8, 136.7)
- moved R4 36.7 mm to (180.1, 134.1), turned to 180 degrees
- moved J1 35.7 mm to (185.6, 142.4), turned to 180 degrees
- moved R8 34.4 mm to (180.1, 132.6), turned to 0 degrees
- moved J4 34.4 mm to (184.0, 127.0), turned to -90 degrees
- moved J3 32.9 mm to (184.0, 112.7), turned to -90 degrees
- moved C6 32.3 mm to (177.7, 132.6), turned to -90 degrees
- moved Q7 31.0 mm to (175.7, 132.9), turned to 90 degrees
- moved D2 30.3 mm to (180.1, 108.9), turned to 0 degrees
- moved G*** 29.8 mm to (163.1, 109.1), turned to 180 degrees
- moved U8 29.8 mm to (173.2, 133.2), turned to 0 degrees
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Routing:
- net VCC: track 33.1 -> 62.1 mm
- net Net-(Q7-G): track 11.1 -> 4.38 mm
- net Net-(Q8-G): track 9.27 -> 2.82 mm
- net Net-(D3-K): track 4.31 -> 0.00 mm
- net Net-(U8-LO): track 3.68 -> 1.56 mm
- net GNDS: track 8.45 -> 7.88 mm
- net ch1_1: track 3.77 -> 3.55 mm, vias 1 -> 0
- removed copper zone on F.Cu, net VCC
Other:
- board size 51.2 x 29.8 mm -> 44.7 x 51.4 mm
- copper layers 2 -> 4

Commit message: a
Parts:
- added J5: Conn_01x05_Pin, Connector_PinSocket_2.54mm:PinSocket_1x05_P2.54mm_Vertical, F.Cu at (226.8, 119.6)
- added J6: Conn_01x05_Pin, Connector_PinSocket_2.54mm:PinSocket_1x05_P2.54mm_Vertical, F.Cu at (231.4, 119.6)
- added J7: Conn_01x04_Pin, Connector_PinSocket_2.54mm:PinSocket_1x04_P2.54mm_Vertical, F.Cu at (164.4, 146.1)
- C3, C5: moved to B.Cu
- moved U2 31.6 mm to (136.4, 124.8), turned to 0 degrees
- moved U10 28.5 mm to (139.6, 141.6)
- moved U9 24.3 mm to (141.6, 132.1), turned to 0 degrees
- moved C3 16.7 mm to (152.1, 118.1)
- moved U6 9.17 mm to (176.2, 113.1), turned to 90 degrees
- moved C5 9.08 mm to (159.8, 108.2)
- moved C4 7.29 mm to (184.5, 113.8)
- moved R10 7.29 mm to (186.9, 129.3)
- moved C2 7.29 mm to (184.5, 127.7)
- moved C6 7.29 mm to (184.5, 135.2)
- moved C8 7.29 mm to (184.5, 119.6)
- moved D1 7.29 mm to (186.1, 125.2)
- moved D2 7.29 mm to (186.9, 111.5)
- moved D3 7.29 mm to (185.0, 131.9)
- moved D4 7.29 mm to (186.9, 117.2)
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Connections:
- C23 pad 1: VDD -> +3V3
- J2 pad 1: unconnected-(J2-Pin_1-Pad1) -> GND1
- J2 pad 2: unconnected-(J2-Pin_2-Pad2) -> +3V3
- J2 pad 4: unconnected-(J2-Pin_4-Pad4) -> +5V
- J2 pad 6: unconnected-(J2-Pin_6-Pad6) -> LED1
- J2 pad 7: unconnected-(J2-Pin_7-Pad7) -> TX
- J2 pad 9: unconnected-(J2-Pin_9-Pad9) -> RX
- U10 pad 18: unconnected-(U10-PA13-Pad18) -> DIO
- U10 pad 19: unconnected-(U10-PA14-Pad19) -> cLK
- U10 pad 4: VDD -> +3V3
- U2 pad 1: VDD -> +5V
- U2 pad 2: unconnected-(U2-INA-Pad2) -> PWM2_1
- U2 pad 3: unconnected-(U2-INB-Pad3) -> PWM2_2
- U4 pad 10: VDDA -> +3V3
- U4 pad 3: GNDS -> GND1
- U6 pad 1: GND -> Net-(Q4-S)
- U6 pad 10: VDDA -> +3V3
- U6 pad 2: Net-(Q4-S) -> GND
- U6 pad 3: GNDS -> GND1
- U9 pad 1: VDD -> +5V
- U9 pad 2: unconnected-(U9-INA-Pad2) -> PWM1_1
- U9 pad 3: unconnected-(U9-INB-Pad3) -> PWM1_2
Routing:
- net VCC: track 62.1 -> 0.00 mm, vias 2 -> 0
- net GND: track 19.6 -> 0.00 mm
- net Net-(Q1-G): track 9.55 -> 0.00 mm, vias 1 -> 0
- net Net-(Q5-G): track 9.35 -> 0.00 mm, vias 1 -> 0
- net Net-(Q3-G): track 9.06 -> 0.00 mm, vias 1 -> 0
- net GNDS: track 7.88 -> 0.00 mm, vias 2 -> 0
- net VDDA: track 6.25 -> 0.00 mm, vias 2 -> 0
- net Net-(D2-K): track 5.64 -> 0.00 mm
- net Net-(Q7-G): track 4.38 -> 0.00 mm, vias 1 -> 0
- net Net-(D4-K): track 4.29 -> 0.00 mm
- net ch2_2: track 4.03 -> 0.00 mm, vias 1 -> 0
- net Net-(D1-K): track 3.98 -> 0.00 mm
- net Net-(U3-HO): track 3.96 -> 0.00 mm
- net ch1_2: track 3.71 -> 0.00 mm, vias 1 -> 0
- net ch2_1: track 3.69 -> 0.00 mm, vias 1 -> 0
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Other:
- board size 44.7 x 51.4 mm -> 49.3 x 51.4 mm

Commit message: a
Parts:
- U10, U9: moved to F.Cu
- moved U9 30.7 mm to (172.2, 130.0)
- moved U10 30.4 mm to (169.8, 137.7), turned to 0 degrees
Other:
- board size 49.3 x 51.4 mm -> 49.3 x 49.9 mm

Commit message: a
Parts:
- removed C9: C, Capacitor_SMD:C_Elec_10x10.2
- added J8: Conn_01x04_Pin, Connector_PinSocket_2.54mm:PinSocket_1x04_P2.54mm_Vertical, F.Cu at (164.1, 142.9)
- C11, C12, C13, C14, C15, C16, C17, C18, C19, C20, C21, C22, D10, D9, G*** (x2), R19, R20, R21, R22, R23, R24, R25, R26, R28, U5, U9: moved to B.Cu
- C3, C5: moved to F.Cu
- J5, J6: footprint Connector_PinSocket_2.54mm:PinSocket_1x05_P2.54mm_Vertical -> Connector_PinHeader_2.54mm:PinHeader_1x05_P2.54mm_Horizontal
- moved C20 104.4 mm to (182.8, 139.4)
- moved C12 103.0 mm to (184.3, 150.0), turned to 180 degrees
- moved C13 102.5 mm to (170.3, 129.5), turned to -90 degrees
- moved C21 100.2 mm to (177.7, 122.5), turned to -90 degrees
- moved C11 99.3 mm to (191.3, 149.8), turned to 90 degrees
- moved C14 99.2 mm to (175.6, 135.4), turned to -90 degrees
- moved C23 99.1 mm to (174.4, 138.2), turned to 90 degrees
- moved C19 98.1 mm to (191.3, 138.2), turned to -90 degrees
- moved C15 96.8 mm to (180.8, 125.1)
- moved R26 90.3 mm to (186.0, 139.4), turned to 180 degrees
- moved R19 89.4 mm to (188.2, 146.2), turned to -90 degrees
- moved C10 87.9 mm to (169.3, 127.8)
- moved C18 87.8 mm to (182.2, 110.5)
- moved C22 87.1 mm to (191.3, 123.4), turned to -90 degrees
- moved U5 86.2 mm to (188.2, 149.8), turned to 180 degrees
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Connections:
- U10 pad 3: unconnected-(U10-PC15-Pad3) -> LED1
Routing:
- net +5V: track 0.00 -> 68.8 mm, vias 0 -> 2
- net VCC: track 0.00 -> 59.6 mm, vias 0 -> 29
- net Net-(D10-A): track 0.00 -> 37.0 mm, vias 0 -> 3
- net Encoder2_B: track 0.00 -> 34.0 mm, vias 0 -> 1
- net cur_2: track 0.00 -> 32.2 mm, vias 0 -> 2
- net Encoder2_A: track 0.00 -> 26.7 mm, vias 0 -> 1
- net cur_1: track 0.00 -> 26.5 mm, vias 0 -> 2
- net Encoder1_B: track 0.00 -> 21.0 mm, vias 0 -> 1
- net Encoder1_A: track 0.00 -> 18.7 mm, vias 0 -> 1
- net ch1_1: track 0.00 -> 16.5 mm, vias 0 -> 3
- net DIO: track 0.00 -> 15.3 mm, vias 0 -> 1
- net ch2_2: track 0.00 -> 14.7 mm, vias 0 -> 4
- net +3V3: track 0.00 -> 14.5 mm, vias 0 -> 3
- net TX: track 0.00 -> 14.4 mm, vias 0 -> 1
- net Net-(U2-OUTA): track 0.00 -> 14.3 mm, vias 0 -> 1
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- added copper zone on In1.Cu, net +3V3
- added copper zone on In2.Cu, net GND1

Commit message: a
Parts:
- removed C23: C, Capacitor_SMD:C_0603_1608Metric
- added C24: C, Capacitor_SMD:C_0603_1608Metric, B.Cu at (169.9, 152.7)
- added C9: C, Capacitor_SMD:C_Elec_10x10.2, F.Cu at (169.1, 136.6)
- added R29: R, Resistor_SMD:R_0603_1608Metric_Pad0.98x0.95mm_HandSolder, F.Cu at (176.3, 140.0)
- added U11: STM32C092KBT6, Package_QFP:LQFP-32_7x7mm_P0.8mm, B.Cu at (176.0, 152.9)
- U10: value STM32C011F4Px -> BD4104; footprint Package_SO:TSSOP-20_4.4x6.5mm_P0.65mm -> jisaku:SOP-J8; moved to B.Cu
- moved C11 27.1 mm to (168.5, 135.1)
- moved C12 27.1 mm to (161.4, 135.3)
- moved D9 27.1 mm to (166.8, 133.2)
- moved R20 27.1 mm to (168.3, 131.5)
- moved D10 27.1 mm to (163.8, 133.2)
- moved R19 27.1 mm to (165.4, 131.5)
- moved U5 27.1 mm to (165.4, 135.1)
- moved J7 25.1 mm to (161.3, 149.0)
- moved J8 8.51 mm to (164.8, 151.4)
- moved U10 3.42 mm to (172.7, 139.4), turned to 0 degrees
- moved J6 2.03 mm to (164.4, 118.5)
- moved C10 2.01 mm to (169.3, 125.8)
Connections:
- J2 pad 3: unconnected-(J2-Pin_3-Pad3) -> CAN_H
- J2 pad 5: unconnected-(J2-Pin_5-Pad5) -> CAN_L
- U10 pad 1: SCL -> CAN_TX
- U10 pad 2: SDA -> GND1
- U10 pad 3: LED1 -> +5V
- U10 pad 4: +3V3 -> CAN_RX
- U10 pad 5: GND1 -> unconnected-(U10-SPLIT-Pad5)
- U10 pad 6: PWM1_1 -> CAN_L
- U10 pad 7: Encoder2_A -> CAN_H
- U10 pad 8: Encoder2_B -> GND1
Routing:
- net CAN_RX: track 0.00 -> 24.3 mm, vias 0 -> 2
- net Encoder1_B: track 21.0 -> 44.2 mm
- net PWM1_1: track 6.04 -> 27.5 mm, vias 2 -> 0
- net CAN_TX: track 0.00 -> 20.2 mm, vias 0 -> 2
- net Encoder1_A: track 18.7 -> 38.5 mm
- net PWM1_2: track 5.37 -> 24.1 mm, vias 2 -> 0
- net PWM2_1: track 11.8 -> 26.4 mm
- net Encoder2_B: track 34.0 -> 20.8 mm
- net PWM2_2: track 14.0 -> 26.1 mm
- net +3V3: track 14.5 -> 25.9 mm, vias 3 -> 6
- net DIO: track 15.3 -> 26.1 mm
- net cur_2: track 32.2 -> 42.6 mm
- net Net-(D10-A): track 37.0 -> 28.3 mm, vias 3 -> 0
- net CAN_L: track 0.00 -> 8.46 mm, vias 0 -> 1
- net LED1: track 8.34 -> 0.00 mm, vias 1 -> 0
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
Commit message: a
Parts:
- moved R25 3.60 mm to (194.0, 141.0)
- moved C19 0.60 mm to (191.5, 138.7)
- moved R23 0.26 mm to (196.4, 110.8)
Routing:
- net Net-(C21-Pad2): track 11.0 -> 11.9 mm
