File: kicad/MD_mini/MD_mini_v2.kicad_pcb (KiCad board)
At the start: 4 copper layers, 49.3 x 49.9 mm, 91 parts, among them J1 Conn_01x02_Pin, J2 Conn_02x05_Odd_Even, J3 Conn_01x02_Pin, J4 Conn_01x02_Pin, J5 Conn_01x05_Pin, J6 Conn_01x05_Pin, J7 Conn_01x04_Pin, J8 Conn_01x04_Pin, U1 IRS2003, U10 BD4104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

Commit message: a
Parts:
- removed C15, C16, C17, C18, C19, C20, C21, C22: C, Capacitor_SMD:C_0603_1608Metric
- removed R21, R22, R23, R24, R25, R26, R27, R28, R29: R, Resistor_SMD:R_0603_1608Metric_Pad0.98x0.95mm_HandSolder
- removed U10: BD4104, jisaku:SOP-J8
- removed U9: SCM3723ASA, Package_SO:SOIC-8_3.9x4.9mm_P1.27mm
- added C23: 0.1u, Capacitor_SMD:C_0603_1608Metric, B.Cu at (170.8, 130.0)
- added C25: min0.33u, Capacitor_SMD:C_0603_1608Metric, B.Cu at (170.7, 124.4)
- added NJM78L05SU1: ~, jisaku:SOT-89-3, B.Cu at (169.0, 137.6)
- added NJM78L12SU3: ~, jisaku:SOT-89-3, B.Cu at (169.0, 131.7)
- added NJM78L33SU1: ~, jisaku:SOT-89-3, B.Cu at (169.0, 125.8)
- added R43: R, Resistor_SMD:R_0603_1608Metric_Pad0.98x0.95mm_HandSolder, B.Cu at (174.9, 141.9)
- C14: value 0.1u -> min0.33u
- R10, R15, R16, R17, R18: value 10 -> 10k
- R7: value 10 -> 01k
- U2: value SCM3723ASA -> BD4104; footprint Package_SO:SOIC-8_3.9x4.9mm_P1.27mm -> jisaku:SOP-J8
- U5: value ~ -> ADuM1201AR; footprint jisaku:SOT-89-3 -> Package_SO:SOIC-8_3.9x4.9mm_P1.27mm
- moved U2 30.4 mm to (190.2, 148.0), turned to 90 degrees
- moved U5 23.3 mm to (184.7, 148.2), turned to 90 degrees
- moved C12 9.06 mm to (170.0, 132.4), turned to 90 degrees
- moved C13 8.79 mm to (170.0, 138.3), turned to 90 degrees
- moved C11 8.60 mm to (170.0, 126.6)
- moved D10 8.59 mm to (172.4, 133.2), turned to 180 degrees
- moved D9 8.13 mm to (172.5, 139.1), turned to 180 degrees
- moved R20 7.41 mm to (172.4, 137.6), turned to 0 degrees
- moved R19 7.12 mm to (172.5, 131.7), turned to 0 degrees
- moved C14 5.00 mm to (170.7, 136.1), turned to 0 degrees
- moved D1 1.68 mm to (186.0, 125.3), turned to 0 degrees
- moved D2 1.32 mm to (183.4, 110.6), turned to 180 degrees
- turned C1 to 180 degrees
- turned C3 to 180 degrees
- turned C5 to 180 degrees
Connections:
- C1 pad 1: VCC -> Net-(D9-A)
- C11 pad 1: VCC -> Net-(D9-A)
- C12 pad 1: Net-(D10-A) -> VCC
- C13 pad 1: Net-(D10-A) -> Net-(D9-A)
- C14 pad 1: Net-(D10-A) -> +5V
- C24 pad 2: GND1 -> GND
- C3 pad 1: VCC -> Net-(D9-A)
- C5 pad 1: VCC -> Net-(D9-A)
- C7 pad 1: VCC -> Net-(D9-A)
- D10 pad 2: Net-(D10-A) -> VCC
- D9 pad 2: VCC -> Net-(D9-A)
- J2 pad 2: +3V3 -> unconnected-(J2-Pin_2-Pad2)
- J2 pad 4: +5V -> Net-(J2-Pin_4)
- J5 pad 5: GND1 -> GND
- J6 pad 5: GND1 -> GND
- J7 pad 4: GND1 -> GND
- J8 pad 1: GND1 -> GND
- U1 pad 1: VCC -> Net-(D9-A)
- U1 pad 2: Net-(U1-HIN) -> PWM1_1
- U1 pad 3: Net-(U1-HIN) -> PWM1_1
- U11 pad 5: GND1 -> GND
- U2 pad 1: +5V -> Net-(U2-TX)
- U2 pad 2: PWM2_1 -> GND1
- U2 pad 3: PWM2_2 -> Net-(J2-Pin_4)
- U2 pad 4: GND1 -> Net-(U2-RX)
- U2 pad 5: GND -> unconnected-(U2-SPLIT-Pad5)
- U2 pad 6: Net-(U2-OUTB) -> CAN_L
- U2 pad 7: Net-(U2-OUTA) -> CAN_H
- U2 pad 8: Net-(D10-A) -> GND1
- U3 pad 1: VCC -> Net-(D9-A)
- U3 pad 2: Net-(U2-OUTA) -> PWM2_1
- U3 pad 3: Net-(U2-OUTA) -> PWM2_1
- U4 pad 3: GND1 -> GND
- U5 pad 1: Net-(D10-A) -> Net-(J2-Pin_4)
- U5 pad 2: GND -> Net-(U2-TX)
- U5 pad 3: VCC -> Net-(U2-RX)
- U6 pad 3: GND1 -> GND
- U7 pad 1: VCC -> Net-(D9-A)
- U7 pad 2: Net-(U2-OUTB) -> PWM2_2
- U7 pad 3: Net-(U2-OUTB) -> PWM2_2
- U8 pad 1: VCC -> Net-(D9-A)
- U8 pad 2: Net-(U8-HIN) -> PWM1_2
- U8 pad 3: Net-(U8-HIN) -> PWM1_2
Routing:
- net Net-(D9-A): track 0.00 -> 66.3 mm, vias 0 -> 2
- net GND: track 0.16 -> 33.3 mm, vias 42 -> 21
- net Net-(D10-A): track 28.1 -> 0.00 mm
- net GND1: track 9.73 -> 26.7 mm, vias 8 -> 2
- net Net-(J2-Pin_4): track 0.00 -> 16.3 mm, vias 0 -> 1
- net Net-(U2-OUTA): track 15.0 -> 0.00 mm, vias 2 -> 0
- net CAN_RX: track 24.3 -> 10.4 mm, vias 2 -> 0
- net CAN_H: track 4.21 -> 17.9 mm
- net Net-(C21-Pad2): track 11.9 -> 0.00 mm, vias 1 -> 0
- net Encoder1_B: track 44.2 -> 32.6 mm
- net CAN_L: track 8.46 -> 19.8 mm
- net PWM2_1: track 26.4 -> 37.6 mm
- net Net-(U8-HIN): track 9.14 -> 0.00 mm, vias 2 -> 0
- net Net-(U2-TX): track 0.00 -> 8.75 mm
- net Net-(Q2-S): track 8.73 -> 0.00 mm
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