File: kicad/ESC_v1/halfHbridge.kicad_sch (KiCad schematic)
At the start: 15 parts, among them U1 L6389EDTR

Commit message: a
Connections:
- net GND_mech: no longer C1.2, U1.4 (COM)
- new net GND: C1.2, U1.4 (COM)
