File: kicad/ESC_v1/ESC_v1.kicad_pcb (KiCad board)
At the start: 2 copper layers, 148 parts, among them J1 Conn_01x05_Pin, J10 Conn_01x01_Pin, J11 Conn_01x01_Pin, J12 Conn_01x01_Pin, J13 Conn_01x03_Pin, J14 Conn_01x01_Pin, J15 Conn_01x01_Pin, J16 Conn_01x01_Pin, J2 Conn_01x05_Pin, J3 Conn_01x03_Pin, J4 Conn_01x03_Pin, J5 Conn_01x05_Pin, J6 Conn_01x03_Pin, J7 Conn_01x04_Pin, J8 Conn_01x04_Pin, J9 Conn_01x02_Pin, U1 L6389EDTR, U10 BD4104, U19 STM32G431CBUx, U2 L6389EDTR, U3 L6389EDTR, U4 L6389EDTR, U5 L6389EDTR, U6 L6389EDTR, U7 ACS711xEXLT-15AB, U8 ACS711xEXLT-15AB

Commit message: a
Parts:
- added J17: Conn_01x04_Pin, Connector_JST:JST_PH_S4B-PH-K_1x04_P2.00mm_Horizontal, F.Cu at (213.4, 92.8)
- added U11: ADuM1201AR, Package_SO:SOIC-8_3.9x4.9mm_P1.27mm, F.Cu at (242.4, 59.9)
- C1, C10, C11, C12, C17, C18, C2, C21, C22, C5, C6, C9, Q1, Q11, Q3, Q5, Q7, Q9, R1, R10, R13, R14, R15, R16, R19, R2, R20, R25, R26, R28, R31, R32, R34, R4, R7, R8, U1, U10, U19, U2, U3, U4, U5, U6, U7, U8: moved to B.Cu
- J1: footprint Connector_PinSocket_2.54mm:PinSocket_1x05_P2.54mm_Horizontal -> Connector_JST:JST_XH_S5B-XH-A_1x05_P2.50mm_Horizontal; moved to B.Cu
- J2: footprint Connector_PinSocket_2.54mm:PinSocket_1x05_P2.54mm_Horizontal -> Connector_JST:JST_XH_S5B-XH-A_1x05_P2.50mm_Horizontal
- moved J9 137.0 mm to (206.7, 79.6), turned to -90 degrees
- moved J8 136.8 mm to (243.6, 88.5), turned to 90 degrees
- moved C5 124.1 mm to (208.0, 57.4), turned to -90 degrees
- moved U8 121.0 mm to (253.6, 67.8), turned to -90 degrees
- moved U7 119.3 mm to (246.5, 66.5), turned to -90 degrees
- moved C6 116.5 mm to (199.0, 57.8), turned to -90 degrees
- moved J2 116.2 mm to (211.3, 98.3)
- moved R10 116.0 mm to (196.6, 56.6)
- moved J1 116.0 mm to (211.8, 56.7), turned to -90 degrees
- moved U2 115.4 mm to (203.5, 56.5), turned to 180 degrees
- moved J13 114.4 mm to (242.3, 81.2), turned to 180 degrees
- moved R7 114.0 mm to (196.6, 55.1), turned to 180 degrees
- moved R8 113.9 mm to (196.6, 58.2), turned to 180 degrees
- moved R9 112.1 mm to (193.8, 57.8), turned to 180 degrees
- moved C32 110.2 mm to (201.9, 89.8), turned to -90 degrees
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Connections:
- R43 pad 1: CAN_H -> CAN_L
- R43 pad 2: CAN_L -> CAN_H
- U10 pad 1: CAN_TX -> Net-(U10-TX)
- U10 pad 2: GND1 -> Net-(J17-Pin_4)
- U10 pad 3: +5V -> Net-(J17-Pin_1)
- U10 pad 4: CAN_RX -> Net-(U10-RX)
- U10 pad 8: GND1 -> Net-(J17-Pin_4)

Commit message: a
Parts:
- removed C13, C14, C15, C16, C19, C20, C23, C24, C3, C4, C7, C8: C, Capacitor_SMD:C_0603_1608Metric
- removed C34: 1u, Capacitor_SMD:C_0603_1608Metric
- removed D13: LED, LED_SMD:LED_0603_1608Metric
- removed J5: Conn_01x05_Pin, Connector_PinHeader_2.54mm:PinHeader_1x05_P2.54mm_Vertical
- removed J7: Conn_01x04_Pin, Connector_PinSocket_2.54mm:PinSocket_1x04_P2.54mm_Vertical
- removed NJM78L33SU1: ~, jisaku:SOT-89-3
- removed R11, R12, R21, R22, R23, R24, R29, R30, R35, R36, R5, R6: R, Resistor_SMD:R_0603_1608Metric_Pad0.98x0.95mm_HandSolder
- removed TP1, TP10, TP11, TP12, TP2, TP3, TP4, TP5, TP6, TP7, TP8, TP9: TestPoint, TestPoint:TestPoint_THTPad_D1.5mm_Drill0.7mm
- removed U7: ACS711xEXLT-15AB, Sensor_Current:Allegro_QFN-12-10-1EP_3x3mm_P0.5mm
- added NJM78L12SU3: ~, jisaku:SOT-89-3, F.Cu at (199.9, 97.0)
- added R44: 5m, Resistor_SMD:R_2010_5025Metric_Pad1.40x2.65mm_HandSolder, B.Cu at (189.6, 59.3)
- added R45: 5m, Resistor_SMD:R_2010_5025Metric_Pad1.40x2.65mm_HandSolder, B.Cu at (189.6, 65.9)
- added R46: 22, Resistor_SMD:R_0603_1608Metric_Pad0.98x0.95mm_HandSolder, B.Cu at (188.1, 63.6)
- added R47: 22, Resistor_SMD:R_0603_1608Metric_Pad0.98x0.95mm_HandSolder, B.Cu at (188.0, 57.0)
- added R48: R, Resistor_SMD:R_0603_1608Metric_Pad0.98x0.95mm_HandSolder, B.Cu at (191.3, 55.5)
- added R49: R, Resistor_SMD:R_0603_1608Metric_Pad0.98x0.95mm_HandSolder, B.Cu at (191.4, 62.1)
- added R50: R, Resistor_SMD:R_0603_1608Metric_Pad0.98x0.95mm_HandSolder, B.Cu at (191.4, 63.6)
- added R51: 5m, Resistor_SMD:R_2010_5025Metric_Pad1.40x2.65mm_HandSolder, B.Cu at (189.6, 72.3)
- added R52: 22, Resistor_SMD:R_0603_1608Metric_Pad0.98x0.95mm_HandSolder, B.Cu at (188.0, 70.0)
- added R53: R, Resistor_SMD:R_0603_1608Metric_Pad0.98x0.95mm_HandSolder, B.Cu at (191.3, 57.0)
- added R54: R, Resistor_SMD:R_0603_1608Metric_Pad0.98x0.95mm_HandSolder, B.Cu at (191.3, 68.5)
- added R55: R, Resistor_SMD:R_0603_1608Metric_Pad0.98x0.95mm_HandSolder, B.Cu at (191.3, 70.0)
- added U12: ACS711xEXLT-15AB, Sensor_Current:Allegro_QFN-12-10-1EP_3x3mm_P0.5mm, B.Cu at (188.4, 78.2)
- added U9: ACS711xEXLT-15AB, Sensor_Current:Allegro_QFN-12-10-1EP_3x3mm_P0.5mm, B.Cu at (188.6, 84.6)
- C10, C5, J1, Q1, Q11, Q3, Q5, Q7, Q9: moved to F.Cu
- C31, C32, C33, C35, C36, C37, C38, D10, D11, D12, D14, D2, D3, D4, D5, D6, D7, D8, D9, J13, J8, Q10, Q12, Q2, Q4, Q6, Q8, R17, R18, R27, R3, R33, R37, R38, R39, R40, R41, R42, R43, R9, U11: moved to B.Cu
- D1: value D -> LED; footprint Diode_SMD:D_MicroSMP_AK -> LED_SMD:LED_0603_1608Metric; moved to B.Cu
- J10, J11, J12, J14, J15, J16: footprint Connector_Wire:SolderWire-6sqmm_1x01_D3.5mm_OD7mm -> TestPoint:TestPoint_Pad_3.0x3.0mm
- J6: value Conn_01x03_Pin -> Conn_01x06_Pin; footprint Connector_PinHeader_2.54mm:PinHeader_1x03_P2.54mm_Vertical -> Connector_JST:JST_ZH_B6B-ZR_1x06_P1.50mm_Vertical; moved to B.Cu
- moved J6 122.2 mm to (219.0, 68.0), turned to -90 degrees
- moved J3 112.0 mm to (198.8, 61.3), turned to 90 degrees
- moved D14 103.0 mm to (212.8, 85.4), turned to 90 degrees
- moved R43 99.6 mm to (218.4, 101.7), turned to 180 degrees
- moved NJM78L33SU2 97.4 mm to (205.8, 97.0)
- moved NJM78L00SU1 97.4 mm to (194.0, 97.0)
- moved C30 84.3 mm to (206.5, 96.0), turned to 180 degrees
- moved C25 83.9 mm to (200.7, 96.0), turned to 180 degrees
- moved J4 83.9 mm to (173.8, 101.1), turned to 180 degrees
- moved C28 83.4 mm to (204.3, 95.3), turned to 90 degrees
- moved C35 83.4 mm to (216.4, 75.9), turned to -90 degrees
- moved C36 79.8 mm to (214.9, 67.0), turned to 90 degrees
- moved C27 79.1 mm to (198.4, 95.2), turned to 90 degrees
- moved C26 77.5 mm to (194.8, 96.0), turned to 180 degrees
- moved C38 76.8 mm to (212.4, 67.0), turned to 90 degrees
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Connections:
- C1 pad 1: +5V -> +12V
- C1 pad 2: /halfHbridge5/GND_mech -> OPAMP1_VINM0
- C10 pad 1: +5V -> +12V
- C10 pad 2: /halfHbridge4/GND_mech -> OPAMP1_VINM0
- C12 pad 1: Net-(U5-VB) -> Net-(U4-VB)
- C12 pad 2: /halfHbridge4/out1 -> /halfHbridge6/out1
- C17 pad 1: +5V -> +12V
- C17 pad 2: /halfHbridge4/GND_mech -> OPAMP1_VINM0
- C18 pad 1: Net-(U4-VB) -> Net-(U5-VB)
- C21 pad 1: +5V -> +12V
- C21 pad 2: /halfHbridge5/GND_mech -> OPAMP1_VINM0
- C25 pad 1: VCC -> +12V
- C25 pad 2: Net-(NJM78L00SU1-GND) -> OPAMP1_VINM0
- C26 pad 2: Net-(NJM78L00SU1-GND) -> OPAMP1_VINM0
- C27 pad 2: Net-(NJM78L33SU1-GND) -> OPAMP1_VINM0
- C28 pad 1: +3.3V -> +12V
- C28 pad 2: Net-(NJM78L33SU1-GND) -> OPAMP1_VINM0
- C29 pad 1: VCC -> +12V
- C29 pad 2: Net-(NJM78L33SU2-GND) -> OPAMP1_VINM0
- C30 pad 2: Net-(NJM78L33SU2-GND) -> OPAMP1_VINM0
- C31 pad 2: GND -> OPAMP1_VINM0
- C32 pad 2: GND -> OPAMP1_VINM0
- C33 pad 1: +3.3V -> VREF
- C33 pad 2: GND -> OPAMP1_VINM0
- C35 pad 1: +3.3V -> VREF
- C35 pad 2: GND -> OPAMP1_VINM0
- C36 pad 1: +3.3V -> VREF
- C36 pad 2: GND -> OPAMP1_VINM0
- C37 pad 1: +3.3V -> VREF
- C37 pad 2: GND -> OPAMP1_VINM0
- C38 pad 2: GND -> OPAMP1_VINM0
- C5 pad 1: +5V -> +12V
- C5 pad 2: /halfHbridge4/GND_mech -> OPAMP1_VINM0
- C6 pad 2: /halfHbridge6/out1 -> /halfHbridge4/out1
- C9 pad 1: +5V -> +12V
- C9 pad 2: /halfHbridge5/GND_mech -> OPAMP1_VINM0
- D1 pad 1: +3V3 -> /halfHbridge4/out1
- D10 pad 1: /halfHbridge6/out1 -> Net-(D10-K)
- D10 pad 2: Net-(D10-A) -> /halfHbridge6/out1
- D11 pad 1: Net-(D10-A) -> /halfHbridge4/out1
- D11 pad 2: /halfHbridge6/out1 -> Net-(D11-A)
- D12 pad 1: /halfHbridge4/out1 -> Net-(D11-A)
- D12 pad 2: Net-(D12-A) -> /halfHbridge4/out1
- D14 pad 3: Net-(D14-VSS) -> OPAMP1_VINM0
- D8 pad 1: /halfHbridge4/out1 -> Net-(D1-A)
- D8 pad 2: Net-(D8-A) -> /halfHbridge4/out1
- D9 pad 1: Net-(D8-A) -> /halfHbridge6/out1
- D9 pad 2: /halfHbridge4/out1 -> Net-(D10-K)
- J1 pad 5: GND -> OPAMP1_VINM0
- J13 pad 1: Net-(D14-VSS) -> OPAMP1_VINM0
- J2 pad 5: GND -> OPAMP1_VINM0
- J6 pad 1: +5V -> unconnected-(J6-Pin_1-Pad1)
- J6 pad 2: Net-(J5-Pin_1) -> DIO
- J6 pad 3: +3V3 -> CLK
- J8 pad 1: GND -> OPAMP1_VINM0
- J8 pad 2: +3V3 -> VREF
- J9 pad 1: VCC -> OPAMP1_VINM0
- J9 pad 2: GND -> VCC
- NJM78L00SU1 pad 2: Net-(NJM78L00SU1-GND) -> OPAMP1_VINM0
- NJM78L00SU1 pad 3: VCC -> +12V
- NJM78L33SU2 pad 2: Net-(NJM78L33SU2-GND) -> OPAMP1_VINM0
- NJM78L33SU2 pad 3: VCC -> +12V
- Q10 pad 3: /halfHbridge4/GND_mech -> /halfHbridge8/GND_mech
- Q12 pad 3: /halfHbridge5/GND_mech -> /halfHbridge9/GND_mech
- Q3 pad 3: /halfHbridge6/out1 -> /halfHbridge4/out1
- Q4 pad 2: /halfHbridge6/out1 -> /halfHbridge4/out1
- Q6 pad 3: /halfHbridge5/GND_mech -> /halfHbridge7/GND_mech
- Q7 pad 3: /halfHbridge4/out1 -> /halfHbridge6/out1
- Q8 pad 2: /halfHbridge4/out1 -> /halfHbridge6/out1
- Q8 pad 3: /halfHbridge4/GND_mech -> /halfHbridge6/GND_mech
- R10 pad 2: /halfHbridge6/out1 -> /halfHbridge4/out1
- R15 pad 1: Net-(U5-HO) -> Net-(U4-HO)
- R16 pad 1: Net-(U5-LO) -> Net-(U4-LO)
- R17 pad 1: /halfHbridge5/GND_mech -> /halfHbridge7/GND_mech
- R18 pad 1: /halfHbridge4/GND_mech -> /halfHbridge6/GND_mech
- R20 pad 2: /halfHbridge4/out1 -> /halfHbridge6/out1
- R25 pad 1: Net-(U4-HO) -> Net-(U5-HO)
- R26 pad 1: Net-(U4-LO) -> Net-(U5-LO)
- R27 pad 1: /halfHbridge4/GND_mech -> /halfHbridge8/GND_mech
- R33 pad 1: /halfHbridge5/GND_mech -> /halfHbridge9/GND_mech
- R40 pad 1: Net-(D8-A) -> Net-(D1-A)
- R41 pad 1: Net-(D10-A) -> Net-(D10-K)
- R42 pad 1: Net-(D12-A) -> Net-(D11-A)
- U1 pad 3: +5V -> +12V
- U1 pad 4: /halfHbridge5/GND_mech -> OPAMP1_VINM0
- U11 pad 5: GND1 -> OPAMP1_VINM0
- U19 pad 1: +3.3V -> VREF
- U19 pad 11: RX -> OPAMP1_VINM0
- U19 pad 13: TIM2_ETR -> OPAMP1_VINM0
- U19 pad 15: TIM8_CH1N -> OPAMP1_VINP
- U19 pad 16: ADC2_IN5 -> I2C_SCL
- U19 pad 19: ADC2_IN12 -> OPAMP1_VINM0
- U19 pad 21: +3.3V -> VREF
- U19 pad 23: +3.3V -> VREF
- U19 pad 24: ADC1_IN14 -> ADC2_IN14
- U19 pad 25: ADC1_IN11 -> unconnected-(U19-PB12-Pad25)
- U19 pad 26: unconnected-(U19-PB13-Pad26) -> OPAMP3_VINP
- U19 pad 27: SPI_MISO -> OPAMP2_VINP
- U19 pad 28: SPI_MOSI -> ADC2_IN15
- U19 pad 29: TIM8_CH1 -> unconnected-(U19-PC6-Pad29)
- U19 pad 35: +3.3V -> VREF
- U19 pad 38: I2C_SCL -> TIM2_ETR
- U19 pad 39: unconnected-(U19-PC10-Pad39) -> TIM8_CH1N
- U19 pad 42: TIM16_CH1 -> RX
- U19 pad 44: TIM4_CH1 -> TIM8_CH1
- U19 pad 45: I2C_SDA -> unconnected-(U19-PB7-Pad45)
- U19 pad 48: +3.3V -> VREF
- U19 pad 49: GND -> OPAMP1_VINM0
- U19 pad 5: unconnected-(U19-PF0-Pad5) -> I2C_SDA
- U19 pad 6: SPI_SCK -> ADC2_IN10
- U2 pad 1: TIM8_CH2 -> TIM8_CH3
- U2 pad 2: TIM8_CH2N -> TIM8_CH3N
- U2 pad 3: +5V -> +12V
- U2 pad 4: /halfHbridge4/GND_mech -> OPAMP1_VINM0
- U2 pad 6: /halfHbridge6/out1 -> /halfHbridge4/out1
- U3 pad 3: +5V -> +12V
- U3 pad 4: /halfHbridge5/GND_mech -> OPAMP1_VINM0
- U4 pad 1: TIM8_CH3 -> TIM8_CH2
- U4 pad 2: TIM8_CH3N -> TIM8_CH2N
- U4 pad 3: +5V -> +12V
- U4 pad 4: /halfHbridge4/GND_mech -> OPAMP1_VINM0
- U4 pad 6: /halfHbridge8/out1 -> /halfHbridge6/out1
- U5 pad 3: +5V -> +12V
- U5 pad 4: /halfHbridge4/GND_mech -> OPAMP1_VINM0
- U5 pad 6: /halfHbridge4/out1 -> /halfHbridge8/out1
- U6 pad 3: +5V -> +12V
- U6 pad 4: /halfHbridge5/GND_mech -> OPAMP1_VINM0
- U8 pad 1: /halfHbridge4/GND_mech -> /halfHbridge8/GND_mech
- U8 pad 2: GND -> OPAMP1_VINM0
- U8 pad 3: GND -> OPAMP1_VINM0
- U8 pad 9: ADC1_IN14 -> ADC2_IN10
Routing:
- net OPAMP1_VINM0: track 0.00 -> 138.1 mm, vias 0 -> 97
- net VCC: track 0.00 -> 128.5 mm, vias 0 -> 20
- net +5V: track 0.00 -> 105.1 mm, vias 0 -> 1
- net VREF: track 0.00 -> 78.5 mm, vias 0 -> 15
- net +12V: track 0.00 -> 78.3 mm, vias 0 -> 4
- net TIM2_CH1: track 0.00 -> 44.9 mm, vias 0 -> 2
- net TIM2_ETR: track 0.00 -> 42.8 mm, vias 0 -> 1
- net /halfHbridge5/out1: track 0.00 -> 41.7 mm, vias 0 -> 31
- net ADC2_IN15: track 0.00 -> 41.6 mm, vias 0 -> 3
- net /halfHbridge7/out1: track 0.00 -> 40.8 mm, vias 0 -> 31
- net TIM2_CH2: track 0.00 -> 37.2 mm, vias 0 -> 1
- net /halfHbridge9/out1: track 0.00 -> 36.3 mm, vias 0 -> 31
- net OPAMP2_VINP: track 0.00 -> 34.7 mm, vias 0 -> 3
- net ADC2_IN10: track 0.00 -> 34.2 mm, vias 0 -> 3
- net /halfHbridge4/out1: track 0.00 -> 31.3 mm, vias 0 -> 39
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- added copper zone on B.Cu, net /halfHbridge4/GND_mech
- added copper zone on F.Cu, net /halfHbridge4/GND_mech
- added copper zone on F.Cu, net /halfHbridge4/out1
- added copper zone on In1.Cu, net /halfHbridge4/out1
- added copper zone on In2.Cu, net /halfHbridge4/out1
- added copper zone on B.Cu, net /halfHbridge5/GND_mech
- added copper zone on F.Cu, net /halfHbridge5/out1
- added copper zone on In1.Cu, net /halfHbridge5/out1
- added copper zone on In2.Cu, net /halfHbridge5/out1
- added copper zone on B.Cu, net /halfHbridge6/GND_mech
- added copper zone on F.Cu, net /halfHbridge6/GND_mech
- added copper zone on F.Cu, net /halfHbridge6/out1
- added copper zone on In1.Cu, net /halfHbridge6/out1
- added copper zone on In2.Cu, net /halfHbridge6/out1
- added copper zone on B.Cu, net /halfHbridge7/GND_mech
- added copper zone on F.Cu, net /halfHbridge7/out1
- added copper zone on In1.Cu, net /halfHbridge7/out1
- added copper zone on In2.Cu, net /halfHbridge7/out1
- added copper zone on B.Cu, net /halfHbridge8/GND_mech
- added copper zone on F.Cu, net /halfHbridge8/GND_mech
- added copper zone on F.Cu, net /halfHbridge8/out1
- added copper zone on In1.Cu, net /halfHbridge8/out1
- added copper zone on In2.Cu, net /halfHbridge8/out1
- added copper zone on B.Cu, net /halfHbridge9/GND_mech
- added copper zone on F.Cu, net /halfHbridge9/out1
- added copper zone on In1.Cu, net /halfHbridge9/out1
- added copper zone on In2.Cu, net /halfHbridge9/out1
- added copper zone on B.Cu, net OPAMP1_VINM0
- added copper zone on F.Cu, net OPAMP1_VINM0
- added copper zone on In2.Cu, net OPAMP1_VINM0
- added copper zone on F.Cu, net VCC
- added copper zone on In1.Cu, net VREF
Other:
- board outline added: 49.5 x 49.5 mm
- copper layers 2 -> 4

Commit message: a
Connections:
- U19 pad 45: unconnected-(U19-PB7-Pad45) -> TIM4_CH1
Routing:
- net TIM4_CH1: track 0.00 -> 8.91 mm, vias 0 -> 2
- net TIM8_CH2: track 12.4 -> 13.2 mm
