File: kicad/ESC_v1/ESC_v1.kicad_sch (KiCad schematic)
At the start: 41 parts, among them J1 Conn_01x05_Pin, J10 Conn_01x01_Pin, J11 Conn_01x01_Pin, J12 Conn_01x01_Pin, J13 Conn_01x03_Pin, J14 Conn_01x01_Pin, J15 Conn_01x01_Pin, J16 Conn_01x01_Pin, J17 Conn_01x02_Pin, J2 Conn_01x05_Pin, J3 Conn_01x03_Pin, J4 Conn_01x03_Pin, J5 Conn_01x05_Pin, J6 Conn_01x03_Pin, J7 Conn_01x04_Pin, J8 Conn_01x04_Pin, J9 Conn_01x02_Pin, U10 BD4104, U19 STM32G431CBUx, U7 ACS711xEXLT-15AB, U8 ACS711xEXLT-15AB

Commit message: a
Parts:
- removed J17: Conn_01x02_Pin, symbol Connector:Conn_01x02_Pin
- added J17: Conn_01x04_Pin, Connector_JST:JST_PH_S4B-PH-K_1x04_P2.00mm_Horizontal, symbol Connector:Conn_01x04_Pin
- added U11: ADuM1201AR, Package_SO:SOIC-8_3.9x4.9mm_P1.27mm, symbol Isolator:ADuM1201AR
- J1, J2: footprint Connector_PinSocket_2.54mm:PinSocket_1x05_P2.54mm_Horizontal -> Connector_JST:JST_XH_S5B-XH-A_1x05_P2.50mm_Horizontal
Connections:
- net +5V: now also U11.8 (VDD2); no longer U10.3 (VCC)
- net CAN_H: now also R43.2, J17.2 (Pin_2); no longer R43.1
- net CAN_L: now also R43.1, J17.3 (Pin_3); no longer R43.2
- net CAN_RX: now also U11.6 (VOB); no longer U10.4 (RX)
- net CAN_TX: now also U11.7 (VIA); no longer U10.1 (TX)
- net GND1: now also U11.5 (GND2); no longer U10.2 (GND), U10.8 (STB)
- new net: J17.1 (Pin_1), U10.3 (VCC), U11.1 (VDD1)
- new net: U10.1 (TX), U11.2 (VOA)
- new net: U10.4 (RX), U11.3 (VIB)
- new net: J17.4 (Pin_4), U10.2 (GND), U10.8 (STB), U11.4 (GND1)
Other:
- moved on the sheet: C31, C32, C33, C34, C35, C36, C37, C38, J9, R43, U10

Commit message: a
Parts:
- removed D1: D, Diode_SMD:D_MicroSMP_AK, symbol Device:D
- removed J5: Conn_01x05_Pin, Connector_PinHeader_2.54mm:PinHeader_1x05_P2.54mm_Vertical, symbol Connector:Conn_01x05_Pin
- removed J6: Conn_01x03_Pin, Connector_PinHeader_2.54mm:PinHeader_1x03_P2.54mm_Vertical, symbol Connector:Conn_01x03_Pin
- removed J7: Conn_01x04_Pin, Connector_PinSocket_2.54mm:PinSocket_1x04_P2.54mm_Vertical, symbol Connector:Conn_01x04_Pin
- removed J9: Conn_01x02_Pin, Connector_AMASS:AMASS_XT30PW-M_1x02_P2.50mm_Horizontal, symbol Connector:Conn_01x02_Pin
- removed U7: ACS711xEXLT-15AB, Sensor_Current:Allegro_QFN-12-10-1EP_3x3mm_P0.5mm, symbol Sensor_Current:ACS711xEXLT-15AB
- added J5: Conn_01x01_Pin, Connector_Wire:SolderWire-0.75sqmm_1x01_D1.25mm_OD2.3mm, symbol Connector:Conn_01x01_Pin
- added J6: Conn_01x06_Pin, Connector_JST:JST_ZH_B6B-ZR_1x06_P1.50mm_Vertical, symbol Connector:Conn_01x06_Pin
- added R44, R45, R51: 5m, Resistor_SMD:R_2010_5025Metric_Pad1.40x2.65mm_HandSolder, symbol Device:R
- added R46, R47, R52: 22, Resistor_SMD:R_0603_1608Metric_Pad0.98x0.95mm_HandSolder, symbol Device:R
- added R48, R49, R50, R53, R54, R55: R, Resistor_SMD:R_0603_1608Metric_Pad0.98x0.95mm_HandSolder, symbol Device:R
- added U12, U9: ACS711xEXLT-15AB, Sensor_Current:Allegro_QFN-12-10-1EP_3x3mm_P0.5mm, symbol Sensor_Current:ACS711xEXLT-15AB
- J10, J11, J12, J14, J15, J16: footprint Connector_Wire:SolderWire-6sqmm_1x01_D3.5mm_OD7mm -> TestPoint:TestPoint_Pad_3.0x3.0mm
- renumbered NJM78L33SU1 to NJM78L12SU3
Connections:
- net +3V3 is gone; now on net +3.3V: J8.2 (Pin_2)
- net ADC2_IN12 is gone; now on net GND: U19.19 (PB2)
- net ADC2_IN5 is gone; now on net I2C_SCL: U19.16 (PC4)
- net GND1 is gone; now on net GND: U11.5 (GND2)
- net SPI_SCK is gone; now on net ADC2_IN10: U19.6 (PF1)
- net TIM16_CH1 is gone; now on net RX: U19.42 (PB4)
- net VREF is gone; now on net +3.3V: C30.1, C38.1, J3.3 (Pin_3), J4.3 (Pin_3), NJM78L33SU2.1 (Vout), U19.20 (VREF+), U8.10 (VCC)
- net +3.3V: now also R48.1, R49.1, R54.1, U12.10 (VCC), U9.10 (VCC); no longer C28.1, NJM78L12SU3.1 (Vout)
- net CLK: now also J6.3 (Pin_3)
- net DIO: now also J6.2 (Pin_2)
- net GND: now also C25.2, C26.2, C27.2, C28.2, C29.2, C30.2, D14.3 (VSS), J13.1 (Pin_1), NJM78L00SU1.2 (GND), NJM78L12SU3.2 (GND), NJM78L33SU2.2 (GND), U19.11 (PA3), U19.13 (PA5), J5.1 (Pin_1), J6.4 (Pin_4), R44.2, R45.2, R50.2, R51.2, R53.2, R55.2, U12.2 (IP-), U12.3 (GND), U9.2 (IP-), U9.3 (GND)
- net I2C_SCL: no longer U19.38 (PA15)
- net I2C_SDA: now also U19.5 (PF0); no longer U19.45 (PB7)
- net RX: now also J6.6 (Pin_6); no longer U19.11 (PA3)
- net TIM2_ETR: now also U19.38 (PA15); no longer U19.13 (PA5)
- net TIM4_CH1: no longer U19.44 (PB6)
- net TIM8_CH1: now also U19.44 (PB6); no longer U19.29 (PC6)
- net TIM8_CH1N: now also U19.39 (PC10); no longer U19.15 (PA7)
- net TX: now also J6.5 (Pin_5)
- net VCC: no longer C25.1, C29.1, NJM78L00SU1.3 (Vin), NJM78L33SU2.3 (Vin)
- net halfHbridge4/GND_mech: now also U12.1 (IP+); no longer U8.1 (IP+)
- net halfHbridge5/GND_mech: now also R51.1, R52.1
- net OPAMP3_VINP: now reaches U19.26 (PB13)
- net OPAMP3_VINP: now also R52.2, R54.2, R55.1
- net ADC1_IN11: no longer names the net of U19.25 (PB12)
- net ADC1_IN14 renamed ADC2_IN10
- net ADC2_IN10: no longer U19.24 (PB11)
- net SPI_MISO renamed OPAMP2_VINP
- net OPAMP2_VINP: now also R46.2, R49.2, R50.1
- net SPI_MOSI renamed ADC2_IN15
- net ADC2_IN15: now also U9.9 (VIOUT)
- new net +12V: C25.1, C28.1, C29.1, NJM78L00SU1.3 (Vin), NJM78L12SU3.1 (Vout), NJM78L33SU2.3 (Vin)
- new net ADC2_IN14: U12.9 (VIOUT), U19.24 (PB11)
- new net OPAMP1_VINP: R47.2, R48.2, R53.1, U19.15 (PA7)
- new net halfHbridge6/GND_mech: U9.1 (IP+)
- new net halfHbridge7/GND_mech: R45.1, R46.1
- new net halfHbridge8/GND_mech: U8.1 (IP+)
- new net halfHbridge9/GND_mech: R44.1, R47.1
Other:
- moved on the sheet: C31, C32, C38, J14, J15, J16, J17, R43, U10, U11, U8

Commit message: a
Connections:
- net TIM4_CH1: now also U19.45 (PB7)
Changed lines of the file:
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@@
+		)
+	)
+	(global_label "TIM4_CH1"
+		(shape input)
+		(at 180.34 107.95 180)
+		(fields_autoplaced yes)
+		(effects
+			(font
+				(size 1.27 1.27)
+			)
+			(justify right)
+		)
+		(property "Intersheetrefs" "${INTERSHEET_REFS}"
+			(at 168.3439 107.95 0)
+			(effects
+				(font
+					(size 1.27 1.27)
+				)
+				(justify right)
+				(hide yes)
+			)
 		)
 	)
