File: kicad/md_v3/md_v3/md_v3.kicad_pcb (KiCad board)
At the start: 4 copper layers, 49.3 x 49.9 mm, 91 parts, among them J1 Conn_01x02_Pin, J10 Conn_01x02_Pin, J11 Conn_01x02_Pin, J2 Conn_01x05_Pin, J3 Conn_01x03_Pin, J4 Conn_01x02_Pin, J5 Conn_02x05_Odd_Even, J6 Conn_01x06_Pin, J7 Conn_01x05_Pin, J9 Conn_01x03_Pin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

Commit message: a
Parts:
- removed C15: 1u, Capacitor_SMD:C_0603_1608Metric
- removed C20, C21: 0.1u, Capacitor_SMD:C_0603_1608Metric
- removed C22: 330u, Capacitor_SMD:C_Elec_10x10.2
- J9: moved to B.Cu
- moved JP2 30.7 mm to (180.3, 84.7)
- moved JP1 25.3 mm to (185.0, 84.7)
- moved U11 22.8 mm to (183.5, 80.0), turned to 0 degrees
- moved U10 18.6 mm to (191.0, 84.7), turned to 0 degrees
- moved R43 14.7 mm to (192.1, 92.9)
- moved C10 12.1 mm to (206.5, 95.9)
- moved C12 12.1 mm to (203.8, 96.5)
- moved C13 12.1 mm to (201.4, 95.8)
- moved C9 12.1 mm to (208.8, 96.6)
- moved NJM78L05SU1 12.1 mm to (208.0, 97.6)
- moved NJM78L12SU2 12.1 mm to (203.0, 97.5)
- moved NJM78L33SU1 10.6 mm to (196.5, 97.8)
- moved C11 10.6 mm to (195.0, 96.1)
- moved C14 10.6 mm to (197.4, 96.8)
- moved C7 9.73 mm to (188.8, 93.0), turned to 180 degrees
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Routing:
- net VCC: track 3.15 -> 87.1 mm, vias 0 -> 8
- net +3.3V: track 41.7 -> 117.7 mm, vias 3 -> 5
- net +5V: track 22.7 -> 98.6 mm, vias 1 -> 2
- net GNDA: track 18.8 -> 75.9 mm, vias 0 -> 1
- net +12V: track 32.1 -> 75.6 mm, vias 3 -> 6
- net GND: track 17.6 -> 57.3 mm, vias 1 -> 41
- net ch2_2: track 7.36 -> 42.6 mm, vias 0 -> 2
- net C_RX_A: track 6.87 -> 37.2 mm, vias 0 -> 2
- net ch1_1: track 12.8 -> 40.2 mm, vias 0 -> 3
- net ch1_2: track 10.8 -> 38.2 mm, vias 0 -> 1
- net RX: track 43.1 -> 18.3 mm, vias 1 -> 0
- net Net-(Q3-G): track 0.00 -> 24.6 mm, vias 0 -> 3
- net Net-(Q2-G): track 2.62 -> 26.6 mm
- net Net-(Q1-G): track 8.27 -> 29.9 mm, vias 1 -> 2
- net Net-(Q5-G): track 0.00 -> 21.2 mm, vias 0 -> 2
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- added copper zone on B.Cu, net GND
- added copper zone on F.Cu, net GND
- added copper zone on In2.Cu, net GND
- added copper zone on B.Cu, net GND1
- added copper zone on F.Cu, net GND1
- added copper zone on In1.Cu, net GND1
- added copper zone on In2.Cu, net GND1
- added copper zone on B.Cu, net GND2
- added copper zone on F.Cu, net GND2
- added copper zone on In1.Cu, net GND2
- added copper zone on In2.Cu, net GND2
- added copper zone on B.Cu, net VCC
- added copper zone on B.Cu, net ch1_1
- added copper zone on F.Cu, net ch1_1
- added copper zone on In1.Cu, net ch1_1
- added copper zone on In2.Cu, net ch1_1
- added copper zone on B.Cu, net ch1_2
- added copper zone on F.Cu, net ch1_2
- added copper zone on In1.Cu, net ch1_2
- added copper zone on In2.Cu, net ch1_2
- added copper zone on B.Cu, net ch2_1
- added copper zone on F.Cu, net ch2_1
- added copper zone on In1.Cu, net ch2_1
- added copper zone on In2.Cu, net ch2_1
- added copper zone on B.Cu, net ch2_2
- added copper zone on F.Cu, net ch2_2
- added copper zone on In1.Cu, net ch2_2
- added copper zone on In2.Cu, net ch2_2
